File: i2current.kicad_sch (KiCad schematic)
At the start: 98 parts, among them J10 QWIIC, J11 QWIIC, J2 USB_C_Receptacle_USB2.0, J3 CONN_BATT, J4 BIG_OUT, J5 EXT_IFACE, J6 Conn_01x10, J8 Conn_01x06, J9 Conn_01x06, Q1 AO3400A, Q4 AO3400A, Q5 AO3400A, Q6 AO3400A, Q8 AO3400A, SW3 B2, SW4 B2, SW6 SW_SPDT, U10 SMTSO3030CTJ, U11 TPS56637RPAR, U2 SMTSO3030CTJ, U3 SMTSO3030CTJ, U4 TPS5430DDA, U5 FUSB302B01MPX, U8 BQ25792RQMR, U9 SMTSO3030CTJ

Commit message: backup 2
Parts:
- removed R2: 3k, Resistor_SMD:R_0402_1005Metric, symbol Device:R_Small
- added D4, D5: LED, LED_SMD:LED_0603_1608Metric, symbol Device:LED
- added R25, R26, R27: 6k/0603, Resistor_SMD:R_0603_1608Metric_Pad0.98x0.95mm_HandSolder, symbol Device:R_Small
- added TP1: TestPoint, TestPoint:TestPoint_Pad_D1.0mm, symbol Connector:TestPoint
- D1: value LED_0603 -> LED; footprint LED_SMD:LED_0603_1608Metric_Pad1.05x0.95mm_HandSolder -> LED_SMD:LED_0603_1608Metric
- R17: value 3k -> 6k/0603; footprint Resistor_SMD:R_0402_1005Metric -> Resistor_SMD:R_0603_1608Metric_Pad0.98x0.95mm_HandSolder
- R19: value 3k -> 6k/0603
- R22: value 450 -> DNP; footprint Resistor_SMD:R_0402_1005Metric -> Resistor_SMD:R_0603_1608Metric_Pad0.98x0.95mm_HandSolder
- R9: value 10k -> 6k/0603; footprint Resistor_SMD:R_0201_0603Metric -> Resistor_SMD:R_0603_1608Metric_Pad0.98x0.95mm_HandSolder
Connections:
- net +3.3V: now also D5.2 (A)
- net +5V: now also D4.2 (A)
- net +BATT: now also D2.2 (A)
- net 5V_ENA: now also R25.1
- net GLOB_~{OFF}: now also R25.2; no longer D2.2 (A)
- net GND: now also R9.2, U3.1, R26.2, R27.2; no longer R9.1
- net at D2.1 (K): now also R9.1; no longer R9.2
- net at U11.4 (PG): now also TP1.1
- new net: D5.1 (K), R27.1
- new net: D4.1 (K), R26.1
Other:
- note added: "EN thereshold: 0.5V"
- note added: "EN thereshold: 1.18V (1uA current source)"
- note added: "TODO check mosfet"
- moved on the sheet: C10, C22, C23, C24, C25, C26, C27, C28, C3, C4, C41, C42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

Commit message: unratnestd'd
Parts:
- removed C42: 10u, Capacitor_SMD:C_0603_1608Metric, symbol Device:C_Small
- removed R27: 6k/0603, Resistor_SMD:R_0603_1608Metric_Pad0.98x0.95mm_HandSolder, symbol Device:R_Small
- added R2: 3k, Resistor_SMD:R_0402_1005Metric, symbol Device:R_Small
- C23, C24, C28, C3: value 22uF -> 22uF/6.3V
- C41: value 10u -> 22uF/6.3V
- R1, R3: footprint Resistor_SMD:R_0201_0603Metric -> Resistor_SMD:R_0402_1005Metric
- R26: value 6k/0603 -> 3k; footprint Resistor_SMD:R_0603_1608Metric_Pad0.98x0.95mm_HandSolder -> Resistor_SMD:R_0402_1005Metric
- R9: value 6k/0603 -> 10k; footprint Resistor_SMD:R_0603_1608Metric_Pad0.98x0.95mm_HandSolder -> Resistor_SMD:R_0402_1005Metric
Connections:
- net GND: now also R26.1, R9.1, R2.1; no longer R26.2, R9.2
- net at D5.1 (K): now also R2.2
- net at D4.1 (K): now also R26.2; no longer R26.1
- net BQ_SW1: now reaches C20.1, L3.1, U8.28 (SW1)
- net BQ_SW2: now reaches C19.2, L3.2, U8.26 (SW2)
- net at D2.1 (K): now also R9.2; no longer R9.1
Other:
- moved on the sheet: C2, J10, J11, SW4

Commit message: m
Parts:
- added D6, D7: 1N5819WS, Diode_SMD:D_SOD-323, symbol Device:D_Schottky
- added R27, R28: 6k/0603, Resistor_SMD:R_0603_1608Metric_Pad0.98x0.95mm_HandSolder, symbol Device:R_Small
Connections:
- net at Q4.1 (G), Q5.1 (G): now also D6.1 (K), R27.2; no longer U8.10 (ACDRV2)
- net at Q4.2 (S), Q5.2 (S): now also D6.2 (A)
- net at Q1.1 (G), Q8.1 (G): now also D7.1 (K), R28.2; no longer U8.11 (ACDRV1)
- net at Q1.2 (S), Q8.2 (S): now also D7.2 (A)
- new net: R27.1, U8.10 (ACDRV2)
- new net: R28.1, U8.11 (ACDRV1)
Other:
- moved on the sheet: Q1, Q4, Q5, Q8

Commit message: routing 2
Parts:
- removed D1, D4, D5: LED, LED_SMD:LED_0603_1608Metric, symbol Device:LED
- added JP3: VBUS_DC, Jumper:SolderJumper-2_P1.3mm_Open_TrianglePad1.0x1.5mm, symbol Jumper:SolderJumper_2_Open
- added JP4, JP5: USB_CONN, Jumper:SolderJumper-2_P1.3mm_Open_TrianglePad1.0x1.5mm, symbol Jumper:SolderJumper_2_Open
- added LED1, LED2, LED3, LED4: XL-1606UGC, easyeda2kicad:LED-SMD_L1.7-W1.1-R-RD_GREEN, symbol easyeda2kicad:XL-1606UGC
- added R29: 2k, Resistor_SMD:R_0402_1005Metric, symbol Device:R_Small
Connections:
- net GLOB_RST is gone; now on net GLOB_~{OFF}: J8.1 (Pin_1)
- net +3.3V: now also LED2.1 (A)
- net +5V: now also LED1.1 (A)
- net +VDC: now also JP3.1 (A)
- net GLOB_~{OFF}: now also LED4.1 (A)
- net GND: now also DC1.3, R29.2
- net USBIN_M: now also JP5.2 (B); no longer J5.18 (Pin_18)
- net USBIN_P: now also JP4.2 (B); no longer J5.20 (Pin_20)
- net VBUS: now also JP3.2 (B)
- net at R2.2: now also LED2.2 (K)
- net at R26.2: now also LED1.2 (K)
- net 3V3_L: now reaches C8.1, D3.1 (K), L4.2, U4.8 (PH)
- net at U8.1 (STAT): now also LED3.2 (K)
- net at R18.2: now also LED3.1 (A)
- net 5V_L: now reaches C25.2, L1.1, U11.6 (SW)
- new net: LED4.2 (K), R29.1
- new net: J5.18 (Pin_18), JP5.1 (A)
- new net: J5.20 (Pin_20), JP4.1 (A)
Other:
- note added: "@5:78eur, 67.2pln/szt @10:108eur, 46.5pln/szt @20:€171.37, 37pln/szt"
- moved on the sheet: J6, R18
