File: i2current.kicad_sch (KiCad schematic)
At the start: 111 parts, among them J10 QWIIC, J11 QWIIC, J2 USB_C_Receptacle_USB2.0, J3 CONN_BATT, J4 BIG_OUT, J5 EXT_IFACE, J6 Conn_01x10, J8 Conn_01x06, J9 Conn_01x06, Q1 AO3400A, Q4 AO3400A, Q5 AO3400A, Q6 AO3400A, Q8 AO3400A, SW3 B2, SW4 B2, SW6 SW_SPDT, U10 SMTSO3030CTJ, U11 TPS56637RPAR, U2 SMTSO3030CTJ, U3 SMTSO3030CTJ, U4 TPS5430DDA, U5 FUSB302B01MPX, U8 BQ25792RQMR, U9 SMTSO3030CTJ

Commit message: work
Parts:
- removed D2: LED, LED_SMD:LED_0603_1608Metric, symbol Device:LED
- added C15: 22uF/6.3V, Capacitor_SMD:C_0603_1608Metric, symbol Device:C_Small
- added LED5: XL-1606UGC, easyeda2kicad:LED-SMD_L1.7-W1.1-R-RD_GREEN, symbol easyeda2kicad:XL-1606UGC
- added R30: TC33X-2-102E, easyeda2kicad:RES-ADJ-SMD_3P-L3.8-W3.6-P1.90-BL, symbol easyeda2kicad:TC33X-2-102E
- C10: value 100n -> 47p
- C22: value 100n -> 1n
- C4: value 10u -> 22uF/6.3V
- C9: value 100n -> 10n
- R11: value 3k -> 10k
- R14: value 3k -> 2.2k
- R18, R29: value 2k -> 2.2k
Connections:
- net +5V: now also C15.1
- net +BATT: now also J4.3 (Pin_3), LED5.1 (A); no longer J4.1 (Pin_1)
- net +VDC: now also J4.1 (Pin_1); no longer J4.3 (Pin_3)
- net GND: now also C15.2; no longer U10.1, U2.1, U3.1, U9.1
- net at R11.1, U4.5 (VSENSE): now also R30.2, R30.3; no longer R14.2
- net at R9.2: now also LED5.2 (K)
- new net: R14.2, R30.1
Other:
- note added: "3.2k - 3V3 2.2k - 5V"
- moved on the sheet: C41, J1, LED1, R26, U3

Commit message: kinda finish route, needs some checks still
Parts:
- added R31: 10k/DNP, Resistor_SMD:R_0603_1608Metric_Pad0.98x0.95mm_HandSolder, symbol Device:R_Small
Connections:
- net CC1: now also J9.4 (Pin_4); no longer J9.2 (Pin_2)
- net GND: now also U10.1, U2.1, U3.1, U9.1, R31.1
- net LIPO_NTC: now also R31.2
- net USBIN_P: now also J9.2 (Pin_2); no longer J9.4 (Pin_4)
Other:
- note added: "Powernets description: ---------------------- Sinks: +VDC: input from DC Jack or external source (like PoE shield) Sources: +BATT: output from BQ charger - battery packet voltage +VBUS: power from USB - careful, must not assume 5V +3V3: onboard step-down source for ESP32 and stuff, adjustable"
- moved on the sheet: U3

Commit message: i start order
Parts:
- removed J4: BIG_OUT, TerminalBlock_MetzConnect:TerminalBlock_MetzConnect_Type086_RT03406HBLC_1x06_P3.81mm_Horizontal, symbol Connector:Screw_Terminal_01x06
- removed R30: TC33X-2-102E, easyeda2kicad:RES-ADJ-SMD_3P-L3.8-W3.6-P1.90-BL, symbol easyeda2kicad:TC33X-2-102E
- added C42: 10u, Capacitor_SMD:C_0603_1608Metric, symbol Device:C_Small
- added C43, C44: 22uF/6.3V, Capacitor_SMD:C_0603_1608Metric, symbol Device:C_Small
- added CN1: JL15EDGA-38106G01, easyeda2kicad:CONN-TH_6P-P3.81_JILN_JL15EDGA-38106G01, symbol easyeda2kicad:JL15EDGA-38106G01
- added JP6: 5V_ENA, Jumper:SolderJumper-2_P1.3mm_Open_TrianglePad1.0x1.5mm, symbol Jumper:SolderJumper_2_Open
- added R30: 6k/0603, Resistor_SMD:R_0603_1608Metric_Pad0.98x0.95mm_HandSolder, symbol Device:R_Small
- added TP2: TestPoint, TestPoint:TestPoint_Pad_D1.0mm, symbol Connector:TestPoint
- added TP3: WS2812_PIN, TestPoint:TestPoint_THTPad_D1.5mm_Drill0.7mm, symbol Connector:TestPoint
- R14: value 2.2k -> 3k
- R16, R8: value 3k -> 30k
- R20: value 3k -> 100k
- R21: value 3k -> DNP
- R22: value DNP -> 0603/DNP
- R27, R28: value 6k/0603 -> 300/0603
- R31: value 10k/DNP -> 10k/0603/DNP
- R4: value 450 -> 100
- R7: value 3k -> 5k
Connections:
- net +3.3V: now also C43.1, C44.1
- net +BATT: now also CN1.4
- net +VDC: now also CN1.6
- net BAT_IN: now also C42.1, CN1.1
- net BQ_REGN: now also TP2.1
- net GLOB_~{OFF}: now also CN1.5
- net GND: now also C42.2, C43.2, C44.2, CN1.3, R30.1
- net LIPO_NTC: now also CN1.2
- net at R14.2: now also R11.1, U4.5 (VSENSE), JP6.2 (B)
- new net: JP6.1 (A), R30.2
- new net WS2812: TP3.1
- no-connect marks 4 -> 10
Other:
- sheet esp32-c3 ports: added ESP_RX, ESP_TX; removed none
- note added: "Ilim=MAX"
- note added: "Isat=5.7A Iripple = 2.6 Ichg=3A Imax=3+(2.6/2)=4.3A"
- note added: "Powernets description: ---------------------- Sinks: +VDC: input from DC Jack or external source (like PoE shield) Sources: +BATT: output from BQ charger - battery packet voltage +VBUS: power from USB - careful, must not assume 5V +3V3: onboard step-down source for ESP32 and stuff, can be set to 5V"
- note added: "TS (todo next rev) -10;60C"
- note removed: "Powernets description: ---------------------- Sinks: +VDC: input from DC Jack or external source (like PoE shield) Sources: +BATT: output from BQ charger - battery packet voltage +VBUS: power from USB - careful, must not assume 5V +3V3: onboard step-down source for ESP32 and stuff, adjustable"
- note removed: "TODO check mosfet"
- moved on the sheet: C10, C11, C12, C15, C18, C22, C23, C24, C25, C26, C27, C28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

Commit message: 05/24 order
Parts:
- C43: value 22uF/6.3V -> 2u2
- R18, R29: value 2.2k -> 3k
Other:
- note added: "C352437"
- note added: "care, 16V mounted"
- note removed: "BAT: 3.7-4.2V"
- note removed: "ESP32: 3.3V"
- note removed: "OUT: 5V"
- note removed: "VIN: 5-20V"
Changed lines of the file:
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@@
 		)
 	)
-	(polyline
-		(pts
-			(xy -50.8 -8.89) (xy -33.02 -8.89)
-		)
-		(stroke
-			(width 0)
-			(type default)
-		)
-	)
 	(wire
 		(pts
@@
 		)
 	)
-	(text "OUT: 5V"
-		(exclude_from_sim no)
-		(at -29.21 -7.62 0)
-		(effects
-			(font
-				(size 1.27 1.27)
-			)
-			(justify left bottom)
-		)
-	)
 	(text "C393937"
 		(exclude_from_sim no)
@@
 		)
 	)
-	(text "VIN: 5-20V"
-		(exclude_from_sim no)
-		(at -66.04 -7.62 0)
-		(effects
-			(font
-				(size 1.27 1.27)
-			)
-			(justify left bottom)
-		)
-	)
 	(text "Rprog\n1.5MHz settings:\n1S - 3k\n2S - 6.04k\n3S - 10.5k\n4S - 17.4k"
 		(exclude_from_sim no)
@@
 		)
 	)
-	(text "ESP32: 3.3V"
+	(text "Ilim=MAX"
 		(exclude_from_sim no)
-		(at -30.48 2.54 0)
+		(at 145.034 112.522 0)
 		(effects
 			(font
 				(size 1.27 1.27)
 			)
-			(justify left bottom)
+			(justify left)
 		)
 	)
-	(text "Ilim=MAX"
+	(text "care, 16V mounted"
 		(exclude_from_sim no)
-		(at 145.034 112.522 0)
+		(at 70.358 45.974 0)
 		(effects
 			(font
 				(size 1.27 1.27)
 			)
-			(justify left)
 		)
 	)
@@
 		)
 	)
-	(text "BAT: 3.7-4.2V"
+	(text "C352437"
 		(exclude_from_sim no)
-		(at -66.04 7.62 0)
+		(at 96.266 244.856 0)
 		(effects
 			(font
 				(size 1.27 1.27)
 			)
-			(justify left bottom)
 		)
 	)
@@
 			)
 		)
-		(property "Value" "2.2k"
+		(property "Value" "3k"
 			(at 65.405 212.725 0)
 			(effects
@@
 	)
 	(symbol
+		(lib_id "Device:C_Small")
+		(at 99.06 133.35 0)
+		(mirror y)
+		(unit 1)
+		(exclude_from_sim no)
+		(in_bom yes)
+		(on_board yes)
+		(dnp no)
+		(property "Reference" "C43"
+			(at 99.822 135.382 0)
+			(effects
+				(font
+					(size 1.27 1.27)
+				)
+				(justify right)
+			)
+		)
+		(property "Value" "2u2"
+			(at 94.742 135.128 0)
+			(effects
+				(font
+					(size 1.27 1.27)
+				)
+				(justify right)
+			)
+		)
+		(property "Footprint" "Capacitor_SMD:C_0603_1608Metric"
+			(at 99.06 133.35 0)
+			(effects
+				(font
+					(size 1.27 1.27)
+				)
+				(hide yes)
+			)
+		)
+		(property "Datasheet" "~"
+			(at 99.06 133.35 0)
+			(effects
+				(font
+					(size 1.27 1.27)
+				)
+				(hide yes)
+			)
+		)
+		(property "Description" ""
+			(at 99.06 133.35 0)
+			(effects
+				(font
+					(size 1.27 1.27)
+				)
+				(hide yes)
+			)
+		)
+		(pin "1"
+		)
+		(pin "2"
+		)
+		(instances
+			(project "i2current"
+				(path "/5b28c372-d717-46a4-b70a-f55fa1c8ec9b"
+					(reference "C43")
+					(unit 1)
+				)
+			)
+		)
+	)
+	(symbol
 		(lib_id "Device:R_Small")
 		(at 85.09 96.52 180)
@@
 	)
 	(symbol
-		(lib_id "Device:C_Small")
-		(at 99.06 133.35 0)
-		(mirror y)
-		(unit 1)
-		(exclude_from_sim no)
-		(in_bom yes)
-		(on_board yes)
-		(dnp no)
-		(fields_autoplaced yes)
-		(property "Reference" "C43"
-			(at 101.3841 132.6831 0)
-			(effects
-				(font
-					(size 1.27 1.27)
-				)
-				(justify right)
-			)
-		)
-		(property "Value" "22uF/6.3V"
-			(at 101.3841 134.5684 0)
-			(effects
-				(font
-					(size 0.6 0.6)
-				)
-				(justify right)
-			)
-		)
-		(property "Footprint" "Capacitor_SMD:C_0603_1608Metric"
-			(at 99.06 133.35 0)
-			(effects
-				(font
-					(size 1.27 1.27)
-				)
-				(hide yes)
-			)
-		)
-		(property "Datasheet" "~"
-			(at 99.06 133.35 0)
-			(effects
-				(font
-					(size 1.27 1.27)
-				)
-				(hide yes)
-			)
-		)
-		(property "Description" ""
-			(at 99.06 133.35 0)
-			(effects
-				(font
-					(size 1.27 1.27)
-				)
-				(hide yes)
-			)
-		)
-		(pin "1"
-		)
-		(pin "2"
-		)
-		(instances
-			(project "i2current"
-				(path "/5b28c372-d717-46a4-b70a-f55fa1c8ec9b"
-					(reference "C43")
-					(unit 1)
-				)
-			)
-		)
-	)
-	(symbol
 		(lib_id "Device:R_Small")
 		(at 113.03 44.45 270)
@@
 			)
 		)
-		(property "Value" "2.2k"
+		(property "Value" "3k"
 			(at 103.505 89.535 0)
 			(effects

Commit message: start order
Parts:
- removed C24, C28: 22uF/6.3V, Capacitor_SMD:C_0603_1608Metric, symbol Device:C_Small
- removed C7: 100n, Capacitor_SMD:C_0402_1005Metric, symbol Device:C_Small
- removed D3: 1N5819WS, Diode_SMD:D_SOD-323, symbol Device:D_Schottky
- removed J6: Conn_01x10, Connector_Molex:Molex_PicoBlade_53261-1071_1x10-1MP_P1.25mm_Horizontal, symbol Connector_Generic:Conn_01x10
- removed JP2: LIPO_BYPASS, Jumper:SolderJumper-2_P1.3mm_Open_TrianglePad1.0x1.5mm, symbol Jumper:SolderJumper_2_Open
- removed JP5: USB_CONN, Jumper:SolderJumper-2_P1.3mm_Open_TrianglePad1.0x1.5mm, symbol Jumper:SolderJumper_2_Open
- removed JP6: 5V_ENA, Jumper:SolderJumper-2_P1.3mm_Open_TrianglePad1.0x1.5mm, symbol Jumper:SolderJumper_2_Open
- removed L4: FXL0630-6R8-M, easyeda2kicad:IND-SMD_L7.0-W6.6, symbol easyeda2kicad:FXL0630-6R8-M
- removed LED1, LED2, LED3, LED4, LED5: XL-1606UGC, easyeda2kicad:LED-SMD_L1.7-W1.1-R-RD_GREEN, symbol easyeda2kicad:XL-1606UGC
- removed R13: 5.1k/DNP, Resistor_SMD:R_0603_1608Metric_Pad0.98x0.95mm_HandSolder, symbol Device:R_Small
- removed R17, R30: 6k/0603, Resistor_SMD:R_0603_1608Metric_Pad0.98x0.95mm_HandSolder, symbol Device:R_Small
- removed R22: 0603/DNP, Resistor_SMD:R_0603_1608Metric_Pad0.98x0.95mm_HandSolder, symbol Device:R_Small
- removed R26: 3k, Resistor_SMD:R_0402_1005Metric, symbol Device:R_Small
- removed SW3, SW4: B2, Button_Switch_SMD:SW_SPST_TL3342, symbol Switch:SW_Push
- removed U4: TPS5430DDA, Package_SO:SOIC-8_3.9x4.9mm_P1.27mm, symbol Critbit_lib:TPS54331
- added J4: Conn_01x12_MountingPin, Connector_Molex:Molex_PicoBlade_53261-1271_1x12-1MP_P1.25mm_Horizontal, symbol Connector_Generic_MountingPin:Conn_01x12_MountingPin
- added J6: Conn_01x05, Connector_PinHeader_1.27mm:PinHeader_1x05_P1.27mm_Vertical, symbol Connector_Generic:Conn_01x05
- added R33: 75k, Resistor_SMD:R_0402_1005Metric, symbol Device:R_Small
- added R35: 16k, Resistor_SMD:R_0402_1005Metric, symbol Device:R_Small
- added TP4: TestPoint, TestPoint:TestPoint_Pad_D1.0mm, symbol Connector:TestPoint
- added U1: SPX3819M5-L-3-3, Package_TO_SOT_SMD:SOT-23-5, symbol Regulator_Linear:SPX3819M5-L-3-3
- added U12, U13: A-SP1102AR6GHC-A01-2C, easyeda2kicad:LED-SMD_4P-L3.0-W1.5_A-SP1102AR6GHC-A01-2C, symbol easyeda2kicad:A-SP1102AR6GHC-A01-2C
- added U4: FTC252010S4R7MBCA, easyeda2kicad:IND-SMD_L2.5-W2.0-VLS252012CX-150M, symbol easyeda2kicad:FTC252010S4R7MBCA
- added U6: MT2492, easyeda2kicad:SOT-23-6_L2.9-W1.6-P0.95-LS2.8-BL, symbol easyeda2kicad:MT2492
- added U7: ESP32-C3-WROOM-02, Espressif:ESP32-C3-WROOM-02, symbol Espressif:ESP32-C3-WROOM-02
- C10: value 47p -> 10u; footprint Capacitor_SMD:C_0402_1005Metric -> Capacitor_SMD:C_0603_1608Metric
- C22: value 1n -> 10u; footprint Capacitor_SMD:C_0402_1005Metric -> Capacitor_SMD:C_0603_1608Metric
- C23: value 22uF/6.3V -> 10u
- C3: value 22uF/6.3V -> 22n; footprint Capacitor_SMD:C_0603_1608Metric -> Capacitor_SMD:C_0402_1005Metric
- C8: value 100n -> 22uF/6.3V; footprint Capacitor_SMD:C_0402_1005Metric -> Capacitor_SMD:C_0603_1608Metric
- C9: value 10n -> 22uF/6.3V; footprint Capacitor_SMD:C_0402_1005Metric -> Capacitor_SMD:C_0603_1608Metric
- D6, D7: LCSC C191023 -> (none); LCSC Part (none) -> C191023
- J1: value ~ -> B4P
- J8: value Conn_01x06 -> PANEL_CONN
- JP4: value USB_CONN -> 3V3_5V
- R1: value 73.2k -> 75k
- R10: value 5.1k/DNP -> 10k; footprint Resistor_SMD:R_0603_1608Metric_Pad0.98x0.95mm_HandSolder -> Resistor_SMD:R_0402_1005Metric
- R11: value 10k -> 100
- R16: value 30k -> 10k
- R20: value 100k -> 75k
- R25: value 6k/0603 -> 3k; footprint Resistor_SMD:R_0603_1608Metric_Pad0.98x0.95mm_HandSolder -> Resistor_SMD:R_0402_1005Metric
- SW6: LCSC Part (none) -> C393937
- TP3: value WS2812_PIN -> TestPoint; footprint TestPoint:TestPoint_THTPad_D1.5mm_Drill0.7mm -> TestPoint:TestPoint_Pad_D1.0mm
Connections:
- net GLOB_GPIO1 is gone; now on net GND: J5.13 (Pin_13)
- net +3.3V: now also C5.1, C8.1, C9.1, J5.20 (Pin_20), JP4.2 (B), R10.2, R33.2, U4.2, U7.1 (3V3); no longer C11.2, C12.2, C23.1, C3.1, C43.1, C44.1, J5.10 (Pin_10), J5.9 (Pin_9), J8.3 (Pin_3), R11.2, R12.2, R5.2, R6.2, U5.12 (VCONN), U5.13 (VCONN), U5.3 (VDD), U5.4 (VDD)
- net +5V: now also J5.10 (Pin_10), J5.9 (Pin_9), JP4.1 (A), R9.2, J4.12 (Pin_12)
- net +BATT: now also C10.1, C22.1, U1.1 (IN), U1.3 (EN), U6.5 (IN); no longer C5.1
- net 3V3_L: now also C3.1, U4.1, U6.6 (SW); no longer C8.1
- net 5V_ENA: now also R14.1, TP1.1, U7.10 (GPIO10); no longer R25.1
- net BQ_REGN: no longer R18.1, TP2.1, U8.13 (~{CE})
- net CC1: no longer R10.2
- net GLOB_~{OFF}: now also J5.19 (Pin_19), R14.2, R2.2, J4.1 (Pin_1), U12.2 (A); no longer J5.11 (Pin_11), R25.2
- net GND: now also C10.2, C22.2, C8.2, C9.2, R25.1, U8.13 (~{CE}), J4.2 (Pin_2), J4.9 (Pin_9), J4.MP (MountPin), J6.3 (Pin_3), R35.1, TP4.1, U1.2 (GND), U13.3 (K), U13.4 (K), U6.2 (GND), U7.19 (GND), U7.9 (GND); no longer C10.1, C3.2, C9.1, J5.16 (Pin_16), J5.17 (Pin_17), R10.1, R14.1, R16.1, R2.1, R29.2, R9.1
- net I2C_INT: now also J5.14 (Pin_14), J4.6 (Pin_6), U7.3 (GPIO4/ADC1_CH4); no longer J5.8 (Pin_8)
- net SCL: now also J5.18 (Pin_18), J4.8 (Pin_8), U7.6 (GPIO7); no longer J5.14 (Pin_14)
- net SDA: now also J5.16 (Pin_16), J4.7 (Pin_7), U7.7 (GPIO8); no longer J5.12 (Pin_12)
- net USBIN_M: now also J4.11 (Pin_11), U7.13 (GPIO18/USB_D-)
- net USBIN_P: now also J4.10 (Pin_10), U7.14 (GPIO19/USB_D+); no longer JP4.2 (B)
- net VBUS: no longer J5.19 (Pin_19), J5.7 (Pin_7)
- net at R11.1: now also SW6.1 (A); no longer R14.2
- net at R29.1: now also U13.2 (A)
- net 5V_PG: now reaches U11.4 (PG)
- net 5V_PG: now also TP2.1, U7.4 (GPIO5/ADC2_CH0); no longer TP1.1
- net BQ_STAT: now reaches U8.1 (STAT)
- net BQ_STAT: now also R16.1, R18.1
- net at R18.2: now also U12.4 (K)
- net VDD: now reaches R16.2
- net VDD: now also C11.2, C12.2, C23.1, C43.1, C44.1, J8.3 (Pin_3), R11.2, R12.2, R5.2, R6.2, U5.12 (VCONN), U5.13 (VCONN), U5.3 (VDD), U5.4 (VDD), U1.5 (OUT), U12.1 (A); no longer C22.1
- net GLOB_GPIO2 renamed PWRBRD_TX
- net PWRBRD_TX: now also J4.3 (Pin_3), J6.4 (Pin_4), U7.12 (GPIO21/U0TXD)
- net WS2812 renamed 3V3_ENA
- net 3V3_ENA: now also R2.1, U6.4 (EN)
- net esp32-c3/ESP_EN renamed ESP_EN
- net ESP_EN: now also R10.1, J6.1 (Pin_1), U7.2 (EN/CHIP_PU)
- net esp32-c3/IO9 renamed PWRBRD_BOOT
- net PWRBRD_BOOT: now also J5.12 (Pin_12), J4.5 (Pin_5), J6.2 (Pin_2), U7.8 (GPIO9)
- new net: R9.1, U13.1 (A)
- new net: R33.1, R35.2, U6.3 (FB)
- new net: R25.2, U12.3 (K)
- new net: C3.2, U6.1 (BS)
- new net MCU_IO1: J5.7 (Pin_7), U7.17 (GPIO1/ADC1_CH1/XTAL_32K_N)
- new net MCU_IO2: J5.8 (Pin_8), U7.16 (GPIO2/ADC1_CH2)
- new net MCU_IO3: J5.11 (Pin_11), U7.15 (GPIO3/ADC1_CH3)
- new net PWRBRD_RX: J4.4 (Pin_4), J5.17 (Pin_17), J6.5 (Pin_5), U7.11 (GPIO20/U0RXD)
- new net PWRBRD_STAT: R29.2, U7.5 (GPIO6)
- no-connect marks 10 -> 5
Other:
- removed sheet esp32-c3
- note added: "EN thereshold: >1.18V (1uA current source) Vout = 0.6*(1+R1/R2) 0.6* (1+(75k/10k)) Vout = 5.1"
- note added: "EN thereshold: >1.5 R2 = R1/[(Vout/Vfb) - 1] R2 = 75k/[3.3/0.6)-1] R2 = 16.66k = 16k Vout = 3.41"
- note added: "Log 05/24 * Initial release 07/24 TODO: * 5V is now main voltage * 3V3 comes from 5V *"
- note added: "RTS DTR GND PRX PTX"
- note removed: "3.2k - 3V3 2.2k - 5V"
- note removed: "C393937"
- note removed: "C500113"
- note removed: "EN thereshold: 0.5V"
- note removed: "EN thereshold: 1.18V (1uA current source)"
- moved on the sheet: C11, C12, C13, C14, C15, C17, C18, C19, C20, C21, C25, C26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
