File: i2current.kicad_pcb (KiCad board)
At the start: 2 copper layers, 45 x 76 mm, 69 parts, among them J11 Screw_Terminal_01x02, J12 Screw_Terminal_01x02, J2 USB_C_Receptacle_USB2.0, J3 CONN_BATT, J5 EXT_IFACE, J6 Conn_01x10, J7 Conn_01x05, J8 Conn_01x06, J9 Conn_01x06, Q1 AO3400A, Q4 AO3400A, Q5 AO3400A, Q6 AO3400A, Q8 AO3400A, SW2 HARD_RST_BUT, SW3 B2, SW4 B2, SW6 SW_SPDT, U1 TPS61022, U10 SMTSO3030CTJ, U2 SMTSO3030CTJ, U3 SPX3819M5-L-3-3, U5 FUSB302B01MPX, U6 XT30(2+2)PW-M.G.B, U7 ESP32-C3-WROOM-02, U8 BQ25792RQMR, U9 SMTSO3030CTJ

Commit message: do backup kids
Parts:
- removed J12: Screw_Terminal_01x02, TerminalBlock_MetzConnect:TerminalBlock_MetzConnect_Type086_RT03402HBLC_1x02_P3.81mm_Horizontal
- removed SW2: HARD_RST_BUT, Button_Switch_SMD:SW_SPST_TL3342
- removed U1: TPS61022, Package_DFN_QFN:Texas_RWU0007A_VQFN-7_2x2mm_P0.5mm
- removed U6: XT30(2+2)PW-M.G.B, crap:CONN-TH_4P-XT30PW-M
- added C22: 100n, Capacitor_SMD:C_0402_1005Metric, F.Cu at (69.9, 83.7)
- added C23: 22uF, Capacitor_SMD:C_0603_1608Metric, F.Cu at (75.9, 87.2)
- added C24: 22uF, Capacitor_SMD:C_0603_1608Metric, F.Cu at (72.3, 81.5)
- added C25: 100n, Capacitor_SMD:C_0402_1005Metric, F.Cu at (83.5, 70.9)
- added C26: 10u, Capacitor_SMD:C_0603_1608Metric, F.Cu at (77.2, 74.9)
- added C27: 100n, Capacitor_SMD:C_0402_1005Metric, F.Cu at (77.8, 72.0)
- added C28: 22uF, Capacitor_SMD:C_0603_1608Metric, F.Cu at (77.5, 87.2)
- added C29: 2u2, Capacitor_SMD:C_0603_1608Metric, F.Cu at (25.4, 76.0)
- added C30: 2u2, Capacitor_SMD:C_0603_1608Metric, F.Cu at (27.9, 76.0)
- added C31: 10u, Capacitor_SMD:C_0603_1608Metric, F.Cu at (72.9, 68.2)
- added C32: 10u, Capacitor_SMD:C_0603_1608Metric, F.Cu at (71.4, 68.2)
- added C33: 10u, Capacitor_SMD:C_0603_1608Metric, F.Cu at (64.4, 68.3)
- added C34: 10u, Capacitor_SMD:C_0603_1608Metric, F.Cu at (65.9, 68.3)
- added C35: 100n, Capacitor_SMD:C_0402_1005Metric, F.Cu at (67.7, 69.0)
- added C36: 100n, Capacitor_SMD:C_0402_1005Metric, F.Cu at (69.6, 69.0)
- added C37: 10u, Capacitor_SMD:C_0603_1608Metric, F.Cu at (74.6, 68.2)
- added C38: 100n, Capacitor_SMD:C_0402_1005Metric, F.Cu at (65.2, 70.4)
- added C39: 10u, Capacitor_SMD:C_0603_1608Metric, F.Cu at (63.5, 71.4)
- added C40: 10u, Capacitor_SMD:C_0603_1608Metric, F.Cu at (62.0, 71.4)
- added C41: 10u, Capacitor_SMD:C_0603_1608Metric, F.Cu at (84.1, 72.2)
- added C42: 10u, Capacitor_SMD:C_0603_1608Metric, F.Cu at (84.1, 75.2)
- added C5: 10u, Capacitor_SMD:C_0603_1608Metric, F.Cu at (65.2, 83.0)
- added C7: 100n, Capacitor_SMD:C_0402_1005Metric, F.Cu at (63.1, 80.3)
- added C8: 100n, Capacitor_SMD:C_0402_1005Metric, F.Cu at (71.1, 76.2)
- added D3: 1N5819WS, Diode_SMD:D_SOD-323, F.Cu at (72.3, 78.3)
- added J10: QWIIC, Connector_JST:JST_SH_SM04B-SRSS-TB_1x04-1MP_P1.00mm_Horizontal, B.Cu at (100.8, 73.5)
- added J4: BIG_OUT, TerminalBlock_MetzConnect:TerminalBlock_MetzConnect_Type086_RT03406HBLC_1x06_P3.81mm_Horizontal, F.Cu at (57.3, 56.4)
- added JP1: HARDRST, Jumper:SolderJumper-2_P1.3mm_Open_TrianglePad1.0x1.5mm, B.Cu at (64.6, 77.1)
- added L4: FXL0630-6R8-M, easyeda2kicad:IND-SMD_L7.0-W6.6, F.Cu at (76.8, 81.3)
- added R11: 3k, Resistor_SMD:R_0402_1005Metric, F.Cu at (72.0, 83.7)
- added R14: 3k, Resistor_SMD:R_0402_1005Metric, F.Cu at (71.5, 85.1)
- added R16: 3k, Resistor_SMD:R_0402_1005Metric, F.Cu at (69.9, 84.7)
- added R17: 3k, Resistor_SMD:R_0402_1005Metric, F.Cu at (63.0, 88.2)
- added R22: 450, Resistor_SMD:R_0402_1005Metric, F.Cu at (57.3, 111.2)
- added R23: 2, Resistor_SMD:R_0402_1005Metric, F.Cu at (36.8, 72.6)
- added R24: 2, Resistor_SMD:R_0402_1005Metric, F.Cu at (38.8, 72.6)
- added U11: TPS56637RPAR, easyeda2kicad:VQFN-HR-10_L3.0-W3.0_RPA, F.Cu at (80.1, 72.4)
- added U4: TPS5430DDA, Package_SO:SOIC-8_3.9x4.9mm_P1.27mm, F.Cu at (67.4, 79.4)
- C10, C9: value 4.7u -> 100n
- C16, C17, C18, C6: footprint Capacitor_SMD:C_0402_1005Metric -> Capacitor_SMD:C_0603_1608Metric
- C21: value 10u -> 4.7u/10V
- C3: value 4.7u -> 22uF; footprint Capacitor_SMD:C_0402_1005Metric -> Capacitor_SMD:C_0603_1608Metric
- C4: value 4.7u -> 10u; footprint Capacitor_SMD:C_0402_1005Metric -> Capacitor_SMD:C_0603_1608Metric
- J11: value Screw_Terminal_01x02 -> QWIIC; footprint TerminalBlock_MetzConnect:TerminalBlock_MetzConnect_Type086_RT03402HBLC_1x02_P3.81mm_Horizontal -> Connector_JST:JST_SH_SM04B-SRSS-TB_1x04-1MP_P1.00mm_Horizontal; moved to B.Cu
- J7: footprint Connector_PinHeader_1.27mm:PinHeader_1x05_P1.27mm_Vertical -> Critbit_lib:sideclutch
- JP2: moved to B.Cu
- L1: value L -> IHLP3232DZER3R3M11; footprint Inductor_SMD:L_AVX_LMLP07A7 -> easyeda2kicad:IND-SMD_L8.7-W8.2_IHLP-3232CZ
- R1: value 10k -> 73.2k
- R19: footprint Resistor_SMD:R_0402_1005Metric -> Resistor_SMD:R_0603_1608Metric_Pad0.98x0.95mm_HandSolder
- U3: value SPX3819M5-L-3-3 -> SMTSO3030CTJ; footprint Package_TO_SOT_SMD:SOT-23-5 -> easyeda2kicad:SMD_BD5.6-D4.1
- moved D1 43.8 mm to (52.1, 90.9), turned to 0 degrees
- moved R18 42.7 mm to (54.4, 90.8), turned to 90 degrees
- moved D2 41.7 mm to (51.9, 92.6)
- moved R9 38.6 mm to (54.4, 92.6), turned to -90 degrees
- moved C3 36.6 mm to (73.5, 85.9), turned to 180 degrees
- moved J11 33.2 mm to (100.8, 65.8), turned to -90 degrees
- moved R2 32.2 mm to (83.1, 77.5), turned to 0 degrees
- moved R1 29.4 mm to (80.1, 75.3), turned to 0 degrees
- moved R3 28.2 mm to (80.1, 74.6), turned to 180 degrees
- moved C4 27.3 mm to (84.1, 73.7), turned to 180 degrees
- moved J1 27.1 mm to (90.1, 75.4)
- moved L1 25.3 mm to (81.2, 66.2), turned to 0 degrees
- moved J3 23.5 mm to (85.4, 59.0)
- moved C2 21.0 mm to (85.9, 107.7), turned to 180 degrees
- moved C10 17.1 mm to (69.9, 82.6), turned to 180 degrees
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Connections:
- net Net-(J3-Pin_1) renamed /BAT_IN
- net Net-(J3-Pin_2) renamed /LIPO_NTC
- C10 pad 1: +3.3V -> GND
- C10 pad 2: GND -> Net-(U4-COMP)
- C3 pad 1: +BATT -> +3.3V
- C9 pad 1: +BATT -> GND
- C9 pad 2: GND -> Net-(U4-SS)
- D2 pad 2: +BATT -> /GLOB_~{OFF}
- J1 pad 5V: unconnected-(J1-Pad5V) -> +5V
- J1 pad GND: unconnected-(J1-PadGND) -> GND
- J11 pad 1: unconnected-(J11-Pin_1-Pad1) -> GND
- J11 pad 2: unconnected-(J11-Pin_2-Pad2) -> +3.3V
- J5 pad 11: /GLOB_RST -> /GLOB_~{OFF}
- J6 pad 10: /USBIN_P -> /USBIN_M
- J6 pad 9: /USBIN_M -> /USBIN_P
- J7 pad 2: /esp32-c3/IO9/BOOT_BUT1 -> /esp32-c3/IO9
- L1 pad 1: +BATT -> Net-(U11-SW)
- L1 pad 2: Net-(U1-SW) -> +5V
- R2 pad 1: GND -> /5V_ENA
- R2 pad 2: /5V_ENA -> /GLOB_~{OFF}
- SW6 pad 1: unconnected-(SW6-A-Pad1) -> Net-(SW6-A)
- SW6 pad 2: unconnected-(SW6-B-Pad2) -> /GLOB_~{OFF}
- SW6 pad 3: unconnected-(SW6-C-Pad3) -> GND
- U3 pad 1: +BATT -> unconnected-(U3-Pad1)
- U3 pad 2: GND -> (no net)
- U3 pad 3: +BATT -> (no net)
- U3 pad 4: unconnected-(U3-BP-Pad4) -> (no net)
- U8 pad 12: /GLOB_RST -> Net-(JP1-A)
- U8 pad 13: +3.3V -> /BQ_REGN
Routing:
- net +BATT: track 0.00 -> 164.3 mm, vias 0 -> 4
- net +VDC: track 0.00 -> 111.3 mm, vias 0 -> 2
- net VBUS: track 0.00 -> 96.7 mm, vias 0 -> 3
- net GND: track 0.00 -> 69.6 mm, vias 0 -> 14
- net /SDA: track 0.00 -> 60.2 mm, vias 0 -> 6
- net /USBIN_M: track 0.00 -> 55.9 mm, vias 0 -> 2
- net /USBIN_P: track 0.00 -> 55.2 mm, vias 0 -> 2
- net +3.3V: track 0.00 -> 52.5 mm, vias 0 -> 7
- net /LIPO_NTC: track 0.00 -> 51.8 mm, vias 0 -> 2
- net /I2C_INT: track 0.00 -> 51.5 mm, vias 0 -> 8
- net /SCL: track 0.00 -> 41.6 mm, vias 0 -> 5
- net Net-(U8-PROG): track 0.00 -> 30.7 mm, vias 0 -> 2
- net /esp32-c3/ESP_EN: track 0.00 -> 26.8 mm, vias 0 -> 2
- net Net-(Q4-G): track 0.00 -> 20.4 mm, vias 0 -> 2
- net Net-(U8-BATP): track 0.00 -> 18.0 mm, vias 0 -> 2
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- added copper zone on B.Cu, net GND
Other:
- board size 45 x 76 mm -> 47 x 60 mm

Commit message: backup 2
Parts:
- removed R2: 3k, Resistor_SMD:R_0402_1005Metric
- added D4: LED, LED_SMD:LED_0603_1608Metric, F.Cu at (37.4, 107.5)
- added D5: LED, LED_SMD:LED_0603_1608Metric, F.Cu at (37.4, 105.9)
- added R25: 6k/0603, Resistor_SMD:R_0603_1608Metric_Pad0.98x0.95mm_HandSolder, F.Cu at (76.9, 92.8)
- added R26: 6k/0603, Resistor_SMD:R_0603_1608Metric_Pad0.98x0.95mm_HandSolder, F.Cu at (34.1, 107.6)
- added R27: 6k/0603, Resistor_SMD:R_0603_1608Metric_Pad0.98x0.95mm_HandSolder, F.Cu at (34.2, 106.0)
- added TP1: TestPoint, TestPoint:TestPoint_Pad_D1.0mm, B.Cu at (81.6, 74.5)
- D1: value LED_0603 -> LED; footprint LED_SMD:LED_0603_1608Metric_Pad1.05x0.95mm_HandSolder -> LED_SMD:LED_0603_1608Metric
- J10: moved to F.Cu
- J7: footprint Critbit_lib:sideclutch -> Connector_PinHeader_1.27mm:PinHeader_1x05_P1.27mm_Vertical
- R17: value 3k -> 6k/0603; footprint Resistor_SMD:R_0402_1005Metric -> Resistor_SMD:R_0603_1608Metric_Pad0.98x0.95mm_HandSolder
- R19: value 3k -> 6k/0603
- R22: value 450 -> DNP; footprint Resistor_SMD:R_0402_1005Metric -> Resistor_SMD:R_0603_1608Metric_Pad0.98x0.95mm_HandSolder
- R9: value 10k -> 6k/0603; footprint Resistor_SMD:R_0201_0603Metric -> Resistor_SMD:R_0603_1608Metric_Pad0.98x0.95mm_HandSolder
- moved J11 47.1 mm to (83.5, 109.6), turned to 180 degrees
- moved J10 40.0 mm to (83.5, 109.6), turned to 0 degrees
- moved C29 31.8 mm to (53.3, 60.7), turned to 180 degrees
- moved C30 25.6 mm to (53.5, 74.5), turned to 180 degrees
- moved R22 23.7 mm to (35.5, 101.9)
- moved R9 23.4 mm to (34.0, 104.2), turned to 0 degrees
- moved R23 22.4 mm to (56.0, 61.0), turned to 180 degrees
- moved D1 19.3 mm to (33.5, 96.1)
- moved R18 19.2 mm to (35.9, 96.1), turned to 180 degrees
- moved D2 18.7 mm to (37.3, 104.3)
- moved R24 17.3 mm to (56.0, 74.3), turned to 0 degrees
- moved C2 7.58 mm to (79.3, 104.0), turned to -90 degrees
- moved J7 6.52 mm to (81.0, 105.5), turned to 90 degrees
- moved R17 2.75 mm to (60.3, 87.6), turned to 180 degrees
- moved J1 1.35 mm to (91.5, 75.4)
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Connections:
- D2 pad 2: /GLOB_~{OFF} -> +BATT
- R9 pad 1: GND -> Net-(D2-K)
- R9 pad 2: Net-(D2-K) -> GND
- U11 pad 4: unconnected-(U11-PG-Pad4) -> Net-(U11-PG)
- U3 pad 1: unconnected-(U3-Pad1) -> GND
Routing:
- net +VDC: track 111.3 -> 148.9 mm
- net /SCL: track 41.6 -> 68.1 mm, vias 5 -> 6
- net /SDA: track 60.2 -> 83.2 mm, vias 6 -> 7
- net /CC1: track 7.35 -> 26.2 mm, vias 1 -> 4
- net +3.3V: track 52.5 -> 68.9 mm, vias 7 -> 8
- net /I2C_INT: track 51.5 -> 66.9 mm, vias 8 -> 10
- net Net-(U4-EN): track 0.00 -> 12.9 mm, vias 0 -> 2
- net /CC2: track 10.3 -> 22.4 mm, vias 0 -> 1
- net GND: track 69.6 -> 78.9 mm, vias 14 -> 21
- net VBUS: track 96.7 -> 102.7 mm
- net /esp32-c3/TARG_RX: track 12.4 -> 16.8 mm
- net /esp32-c3/TARG_TX: track 11.2 -> 14.3 mm
- net +BATT: track 164.3 -> 167.0 mm
- net /esp32-c3/ESP_EN: track 26.8 -> 29.0 mm, vias 2 -> 1
Other:
- outline, holes or cut-outs redrawn

Commit message: unratnestd'd
Parts:
- removed C42: 10u, Capacitor_SMD:C_0603_1608Metric
- removed R27: 6k/0603, Resistor_SMD:R_0603_1608Metric_Pad0.98x0.95mm_HandSolder
- added R2: 3k, Resistor_SMD:R_0402_1005Metric, F.Cu at (78.9, 106.6)
- C23, C24, C28, C3: value 22uF -> 22uF/6.3V
- C41: value 10u -> 22uF/6.3V
- R1, R3: footprint Resistor_SMD:R_0201_0603Metric -> Resistor_SMD:R_0402_1005Metric
- R26: value 6k/0603 -> 3k; footprint Resistor_SMD:R_0603_1608Metric_Pad0.98x0.95mm_HandSolder -> Resistor_SMD:R_0402_1005Metric
- R9: value 6k/0603 -> 10k; footprint Resistor_SMD:R_0603_1608Metric_Pad0.98x0.95mm_HandSolder -> Resistor_SMD:R_0402_1005Metric
- moved R26 60.1 mm to (84.6, 75.1)
- moved D4 55.9 mm to (84.0, 76.6), turned to 180 degrees
- moved D1 42.6 mm to (63.6, 66.0)
- moved R18 41.8 mm to (63.4, 64.6), turned to 0 degrees
- moved D5 41.5 mm to (78.8, 109.1), turned to -90 degrees
- moved R22 23.3 mm to (57.7, 109.0)
- moved R9 22.5 mm to (55.5, 110.8), turned to 90 degrees
- moved D2 21.4 mm to (57.7, 110.6)
- moved C1 15.2 mm to (60.2, 95.1), turned to -90 degrees
- moved R15 11.8 mm to (60.2, 98.3)
- moved R12 2.45 mm to (69.5, 92.5), turned to 90 degrees
- moved R1 2.24 mm to (82.3, 74.9)
- moved R5 2.19 mm to (68.5, 92.5)
- moved R19 1.60 mm to (63.7, 63.0)
- moved C12 1.55 mm to (67.0, 92.0), turned to 180 degrees
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Connections:
- net Net-(U8-SW1) renamed /BQ_SW1
- net Net-(U8-SW2) renamed /BQ_SW2
- R26 pad 1: Net-(D4-K) -> GND
- R26 pad 2: GND -> Net-(D4-K)
- R9 pad 1: Net-(D2-K) -> GND
- R9 pad 2: GND -> Net-(D2-K)
- U7 pad 10: /esp32-c3/IO10 -> /5V_ENA
- U7 pad 3: /esp32-c3/IO4 -> /I2C_INT
Routing:
- net GND: track 78.9 -> 189.3 mm, vias 21 -> 63
- net /GLOB_~{OFF}: track 0.00 -> 97.6 mm, vias 0 -> 9
- net +3.3V: track 68.9 -> 138.8 mm, vias 8 -> 13
- net +BATT: track 167.0 -> 201.3 mm, vias 4 -> 12
- net /5V_ENA: track 0.00 -> 33.4 mm, vias 0 -> 2
- net +VDC: track 148.9 -> 174.8 mm, vias 2 -> 6
- net /SCL: track 68.1 -> 93.7 mm, vias 6 -> 7
- net /esp32-c3/IO9: track 13.7 -> 37.2 mm, vias 2 -> 4
- net /SDA: track 83.2 -> 104.3 mm, vias 7 -> 6
- net /esp32-c3/ESP_EN: track 29.0 -> 47.1 mm, vias 1 -> 4
- net /I2C_INT: track 66.9 -> 83.5 mm
- net Net-(SW6-A): track 0.00 -> 14.2 mm
- net +5V: track 10.9 -> 20.6 mm
- net VBUS: track 102.7 -> 109.5 mm, vias 3 -> 5
- net /BQ_REGN: track 7.78 -> 11.5 mm, vias 1 -> 3
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- added copper zone on F.Cu, net +VDC
- added copper zone on B.Cu, net /BQ_SW1
- added copper zone on B.Cu, net /BQ_SW2
- added copper zone on F.Cu, net GND
- added copper zone on F.Cu, net VBUS_PIN

Commit message: m
Parts:
- added D6: 1N5819WS, Diode_SMD:D_SOD-323, F.Cu at (37.3, 69.7)
- added D7: 1N5819WS, Diode_SMD:D_SOD-323, F.Cu at (37.3, 72.7)
- added R27: 6k/0603, Resistor_SMD:R_0603_1608Metric_Pad0.98x0.95mm_HandSolder, F.Cu at (41.6, 69.5)
- added R28: 6k/0603, Resistor_SMD:R_0603_1608Metric_Pad0.98x0.95mm_HandSolder, F.Cu at (41.5, 72.6)
- moved JP1 4.53 mm to (69.0, 76.8), turned to 0 degrees
- moved R11 3.20 mm to (73.1, 86.7), turned to -90 degrees
- moved C8 2.11 mm to (72.2, 78.0)
- moved D3 1.90 mm to (72.3, 80.2)
- moved C24 1.80 mm to (72.4, 83.3)
- moved C3 1.44 mm to (74.3, 87.1), turned to -90 degrees
- moved R14 0.92 mm to (72.1, 85.8)
- moved C21 0.67 mm to (69.2, 74.9), turned to 0 degrees
Connections:
- Q1 pad 1: Net-(Q1-G) -> Net-(D7-K)
- Q4 pad 1: Net-(Q4-G) -> Net-(D6-K)
- Q5 pad 1: Net-(Q4-G) -> Net-(D6-K)
- Q8 pad 1: Net-(Q1-G) -> Net-(D7-K)
- U8 pad 10: Net-(Q4-G) -> Net-(U8-ACDRV2)
- U8 pad 11: Net-(Q1-G) -> Net-(U8-ACDRV1)
Routing:
- net Net-(Q4-G): track 19.9 -> 0.00 mm, vias 2 -> 0
- net (no net): track 0.00 -> 19.9 mm, vias 0 -> 2
- net Net-(Q1-G): track 11.7 -> 0.00 mm, vias 2 -> 0
- net Net-(D7-K): track 0.00 -> 9.44 mm, vias 0 -> 1
- net GND: track 189.3 -> 185.9 mm, vias 63 -> 61
- net +3.3V: track 138.8 -> 135.9 mm
- net Net-(D3-K): track 8.42 -> 6.13 mm
- net Net-(JP1-A): track 5.48 -> 3.41 mm
- net Net-(U4-VSENSE): track 4.62 -> 6.58 mm
- net /SDA: track 104.3 -> 106.3 mm
- net Net-(U4-COMP): track 6.49 -> 5.26 mm, vias 2 -> 0
- net /I2C_INT: track 83.5 -> 83.6 mm, vias 10 -> 9

Commit message: routing 2
Parts:
- removed D1, D4, D5: LED, LED_SMD:LED_0603_1608Metric
- added JP3: VBUS_DC, Jumper:SolderJumper-2_P1.3mm_Open_TrianglePad1.0x1.5mm, F.Cu at (60.7, 76.4)
- added JP4: USB_CONN, Jumper:SolderJumper-2_P1.3mm_Open_TrianglePad1.0x1.5mm, B.Cu at (83.4, 100.1)
- added JP5: USB_CONN, Jumper:SolderJumper-2_P1.3mm_Open_TrianglePad1.0x1.5mm, B.Cu at (83.4, 97.6)
- added LED1: XL-1606UGC, easyeda2kicad:LED-SMD_L1.7-W1.1-R-RD_GREEN, F.Cu at (97.0, 76.0)
- added LED2: XL-1606UGC, easyeda2kicad:LED-SMD_L1.7-W1.1-R-RD_GREEN, F.Cu at (58.1, 111.5)
- added LED3: XL-1606UGC, easyeda2kicad:LED-SMD_L1.7-W1.1-R-RD_GREEN, F.Cu at (49.0, 74.2)
- added LED4: XL-1606UGC, easyeda2kicad:LED-SMD_L1.7-W1.1-R-RD_GREEN, F.Cu at (49.0, 87.7)
- added R29: 2k, Resistor_SMD:R_0402_1005Metric, F.Cu at (51.5, 89.1)
- moved D6 33.1 mm to (67.5, 83.3), turned to 180 degrees
- moved R27 29.2 mm to (68.6, 80.5), turned to -90 degrees
- moved D7 27.8 mm to (64.8, 76.4), turned to 90 degrees
- moved R28 25.5 mm to (66.7, 76.4), turned to -90 degrees
- moved R25 21.5 mm to (90.5, 76.8), turned to 0 degrees
- moved C29 19.2 mm to (63.0, 77.3), turned to -90 degrees
- moved C7 16.7 mm to (79.0, 74.6), turned to 180 degrees
- moved R23 15.8 mm to (62.9, 75.2)
- moved C5 15.1 mm to (79.1, 77.0), turned to -90 degrees
- moved R19 14.5 mm to (73.4, 73.8), turned to 0 degrees
- moved C30 13.8 mm to (64.2, 83.2), turned to 0 degrees
- moved R18 13.6 mm to (52.5, 72.7), turned to 180 degrees
- moved R24 13.5 mm to (64.9, 84.5)
- moved C3 13.0 mm to (82.6, 77.0)
- moved R17 11.6 mm to (71.7, 85.3), turned to -90 degrees
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Connections:
- net Net-(D3-K) renamed /3V3_L
- net Net-(U11-SW) renamed /5V_L
- DC1 pad 3: unconnected-(DC1-Pad3) -> GND
- J5 pad 18: /USBIN_M -> Net-(J5-Pin_18)
- J5 pad 20: /USBIN_P -> Net-(J5-Pin_20)
- J8 pad 1: /GLOB_RST -> /GLOB_~{OFF}
Routing:
- net +BATT: track 201.3 -> 41.1 mm, vias 12 -> 14
- net +VDC: track 174.8 -> 66.6 mm, vias 6 -> 8
- net GND: track 185.9 -> 130.6 mm, vias 61 -> 58
- net /GLOB_~{OFF}: track 97.6 -> 47.3 mm, vias 9 -> 6
- net /esp32-c3/ESP_EN: track 47.1 -> 5.54 mm, vias 4 -> 0
- net VBUS: track 109.5 -> 74.0 mm, vias 5 -> 2
- net /esp32-c3/IO9: track 37.2 -> 4.82 mm, vias 4 -> 0
- net /I2C_INT: track 83.6 -> 55.8 mm, vias 9 -> 5
- net /BQ_REGN: track 11.4 -> 33.2 mm, vias 3 -> 4
- net /5V_ENA: track 33.4 -> 12.0 mm, vias 2 -> 1
- net (no net): track 19.9 -> 0.00 mm, vias 2 -> 0
- net Net-(U8-PROG): track 29.1 -> 10.5 mm, vias 2 -> 0
- net /LIPO_NTC: track 51.8 -> 35.7 mm
- net /BAT_IN: track 17.9 -> 2.01 mm
- net /SDA: track 106.3 -> 90.4 mm, vias 6 -> 5
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- added copper zone on F.Cu, net +3.3V
- added copper zone on F.Cu, net +5V
- added copper zone on B.Cu, net +BATT
- added copper zone on F.Cu, net +BATT
- added copper zone on B.Cu, net +VDC
- added copper zone on F.Cu, net /3V3_L
- added copper zone on F.Cu, net /5V_L
- added copper zone on F.Cu, net /BQ_REGN
- added copper zone on B.Cu, net BAT
- added copper zone on F.Cu, net BAT
- added copper zone on B.Cu, net VBUS
Other:
- board size 47 x 60 mm -> 50 x 64 mm
- board text added: "3V3"
- board text added: "5V"
- board text added: "BOOT"
- board text added: "CHG 1-4S"
- board text added: "RST"
- board text added: "USBC-PD"
- board text added: "pwr mux"

Commit message: work
Parts:
- removed D2: LED, LED_SMD:LED_0603_1608Metric
- added LED5: XL-1606UGC, easyeda2kicad:LED-SMD_L1.7-W1.1-R-RD_GREEN, F.Cu at (59.8, 111.4)
- added R30: TC33X-2-102E, easyeda2kicad:RES-ADJ-SMD_3P-L3.8-W3.6-P1.90-BL, F.Cu at (71.8, 85.2)
- C10: value 100n -> 47p
- C15: value 100n -> 22uF/6.3V; footprint Capacitor_SMD:C_0402_1005Metric -> Capacitor_SMD:C_0603_1608Metric
- C22: value 100n -> 1n
- C4: value 10u -> 22uF/6.3V
- C9: value 100n -> 10n
- R11: value 3k -> 10k
- R14: value 3k -> 2.2k
- R18, R29: value 2k -> 2.2k
- moved C15 45.4 mm to (87.4, 71.5)
- moved R2 25.2 mm to (57.1, 110.0), turned to 0 degrees
- moved R6 15.4 mm to (62.6, 99.2)
- moved R5 13.6 mm to (62.1, 97.6), turned to 90 degrees
- moved R12 13.3 mm to (63.1, 97.6), turned to 90 degrees
- moved R26 9.03 mm to (95.7, 76.1), turned to 90 degrees
- moved R9 5.22 mm to (60.6, 109.7), turned to -90 degrees
- moved R17 4.21 mm to (67.5, 85.0), turned to 180 degrees
- moved C10 4.15 mm to (71.8, 77.9), turned to -90 degrees
- moved R16 3.95 mm to (71.8, 76.0), turned to -90 degrees
- moved R15 3.76 mm to (62.1, 94.6), turned to -90 degrees
- moved JP2 3.49 mm to (86.5, 84.4)
- moved C16 3.32 mm to (61.3, 107.0), turned to -90 degrees
- moved R11 3.04 mm to (73.9, 88.7), turned to 0 degrees
- moved C9 2.61 mm to (73.8, 74.4), turned to 180 degrees
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Connections:
- C15 pad 1: +3.3V -> +5V
- J4 pad 1: +BATT -> +VDC
- J4 pad 3: +VDC -> +BATT
- R14 pad 2: Net-(U4-VSENSE) -> Net-(R14-Pad2)
- U10 pad 1: GND -> unconnected-(U10-Pad1)
- U2 pad 1: GND -> unconnected-(U2-Pad1)
- U3 pad 1: GND -> unconnected-(U3-Pad1)
- U9 pad 1: GND -> unconnected-(U9-Pad1)
Routing:
- net +BATT: track 41.1 -> 105.3 mm, vias 14 -> 25
- net /GLOB_~{OFF}: track 47.3 -> 102.7 mm
- net /esp32-c3/ESP_EN: track 5.54 -> 51.7 mm, vias 0 -> 5
- net VBUS: track 74.0 -> 110.6 mm, vias 2 -> 4
- net /esp32-c3/IO9: track 4.82 -> 39.2 mm, vias 0 -> 7
- net /I2C_INT: track 55.8 -> 87.7 mm, vias 5 -> 10
- net /BAT_IN: track 2.01 -> 21.7 mm
- net +3.3V: track 120.9 -> 136.3 mm, vias 11 -> 18
- net /esp32-c3/IO0: track 12.2 -> 0.00 mm
- net /esp32-c3/TARG_RX: track 6.25 -> 18.0 mm, vias 0 -> 1
- net Net-(J5-Pin_18): track 1.22 -> 12.3 mm
- net Net-(J5-Pin_20): track 1.20 -> 12.2 mm
- net /esp32-c3/TARG_TX: track 5.65 -> 15.8 mm, vias 0 -> 1
- net /SCL: track 104.2 -> 94.2 mm, vias 5 -> 8
- net /LIPO_NTC: track 35.7 -> 42.4 mm, vias 2 -> 4
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- added copper zone on B.Cu, net +3.3V
- added copper zone on F.Cu, net /BAT_IN
Other:
- board text added: "3V3-5V"
- board text removed: "3V3"
