File: i2current.kicad_pcb (KiCad board)
At the start: 2 copper layers, 50 x 64 mm, 117 parts, among them J10 QWIIC, J11 QWIIC, J2 USB_C_Receptacle_USB2.0, J3 CONN_BATT, J4 BIG_OUT, J5 EXT_IFACE, J6 Conn_01x10, J7 Conn_01x05, J8 Conn_01x06, J9 Conn_01x06, Q1 AO3400A, Q4 AO3400A, Q5 AO3400A, Q6 AO3400A, Q8 AO3400A, SW3 B2, SW4 B2, SW6 SW_SPDT, U10 SMTSO3030CTJ, U11 TPS56637RPAR, U2 SMTSO3030CTJ, U3 SMTSO3030CTJ, U4 TPS5430DDA, U5 FUSB302B01MPX, U7 ESP32-C3-WROOM-02, U8 BQ25792RQMR, U9 SMTSO3030CTJ

Commit message: kinda finish route, needs some checks still
Parts:
- added R31: 10k/DNP, Resistor_SMD:R_0603_1608Metric_Pad0.98x0.95mm_HandSolder, F.Cu at (78.2, 61.9)
- R10, R13: moved to F.Cu
- moved R10 10.0 mm to (56.5, 72.3), turned to 180 degrees
- moved R13 7.08 mm to (56.2, 89.1), turned to 0 degrees
- moved JP3 0.85 mm to (61.0, 77.2)
- moved R29 0.70 mm to (50.8, 89.1)
- moved JP2 0.55 mm to (86.0, 84.4)
Connections:
- J9 pad 2: /CC1 -> /USBIN_P
- J9 pad 4: /USBIN_P -> /CC1
- U10 pad 1: unconnected-(U10-Pad1) -> GND
- U2 pad 1: unconnected-(U2-Pad1) -> GND
- U3 pad 1: unconnected-(U3-Pad1) -> GND
- U9 pad 1: unconnected-(U9-Pad1) -> GND
Routing:
- net GND: track 135.1 -> 172.4 mm, vias 55 -> 64
- net /5V_ENA: track 10.9 -> 34.6 mm, vias 0 -> 1
- net /GLOB_~{OFF}: track 102.7 -> 125.7 mm, vias 6 -> 7
- net VBUS: track 110.6 -> 91.8 mm, vias 4 -> 10
- net /SDA: track 87.9 -> 103.3 mm, vias 9 -> 10
- net /USBIN_P: track 44.4 -> 50.2 mm
- net /CC1: track 36.6 -> 31.7 mm, vias 4 -> 2
- net +3.3V: track 136.3 -> 140.2 mm, vias 18 -> 20
- net /USBIN_M: track 46.5 -> 50.3 mm, vias 1 -> 3
- net +5V: track 26.8 -> 30.0 mm
- net /BQ_SW2: track 4.93 -> 6.57 mm
- net /esp32-c3/ESP_EN: track 51.7 -> 50.5 mm, vias 5 -> 3
- net /LIPO_NTC: track 42.4 -> 43.6 mm
- net /I2C_INT: track 87.7 -> 88.7 mm
- net /BQ_REGN: track 33.4 -> 34.3 mm
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- added copper zone on F.Cu, net VBUS

Commit message: i start order
Parts:
- removed J4: BIG_OUT, TerminalBlock_MetzConnect:TerminalBlock_MetzConnect_Type086_RT03406HBLC_1x06_P3.81mm_Horizontal
- added C42: 10u, Capacitor_SMD:C_0603_1608Metric, F.Cu at (75.9, 57.8)
- added C43: 22uF/6.3V, Capacitor_SMD:C_0603_1608Metric, F.Cu at (64.7, 88.7)
- added C44: 22uF/6.3V, Capacitor_SMD:C_0603_1608Metric, F.Cu at (70.5, 92.8)
- added CN1: JL15EDGA-38106G01, easyeda2kicad:CONN-TH_6P-P3.81_JILN_JL15EDGA-38106G01, F.Cu at (68.4, 53.3)
- added JP6: 5V_ENA, Jumper:SolderJumper-2_P1.3mm_Open_TrianglePad1.0x1.5mm, F.Cu at (72.1, 83.9)
- added TP2: TestPoint, TestPoint:TestPoint_Pad_D1.0mm, F.Cu at (63.8, 70.4)
- added TP3: WS2812_PIN, TestPoint:TestPoint_THTPad_D1.5mm_Drill0.7mm, F.Cu at (90.1, 74.6)
- R14: value 2.2k -> 3k
- R16, R8: value 3k -> 30k
- R20: value 3k -> 100k
- R21: value 3k -> DNP
- R22: value DNP -> 0603/DNP
- R27, R28: value 6k/0603 -> 300/0603
- R30: value TC33X-2-102E -> 6k/0603; footprint easyeda2kicad:RES-ADJ-SMD_3P-L3.8-W3.6-P1.90-BL -> Resistor_SMD:R_0603_1608Metric_Pad0.98x0.95mm_HandSolder
- R31: value 10k/DNP -> 10k/0603/DNP
- R4: value 450 -> 100
- R7: value 3k -> 5k
- moved R11 1.80 mm to (72.6, 87.4)
- moved R30 0.76 mm to (72.1, 85.9), turned to 180 degrees
- moved R10 0.75 mm to (55.8, 72.3)
- moved J3 0.30 mm to (87.3, 55.5)
- moved JP2 0.30 mm to (85.7, 84.4)
- moved R13 0.20 mm to (56.0, 89.1)
- moved R14 0.20 mm to (71.8, 81.7), turned to 90 degrees
- moved C14 0.12 mm to (63.1, 89.8)
Connections:
- R11 pad 1: Net-(U4-VSENSE) -> Net-(JP6-B)
- R14 pad 2: Net-(R14-Pad2) -> Net-(JP6-B)
- R30 pad 1: Net-(R14-Pad2) -> GND
- R30 pad 2: Net-(U4-VSENSE) -> Net-(JP6-A)
- U4 pad 5: Net-(U4-VSENSE) -> Net-(JP6-B)
- U7 pad 15: /esp32-c3/IO3 -> /GLOB_GPIO2
- U7 pad 16: /esp32-c3/IO2 -> /GLOB_GPIO1
- U7 pad 17: /esp32-c3/IO1 -> /WS2812
Routing:
- net /WS2812: track 0.00 -> 35.0 mm, vias 0 -> 2
- net /GLOB_GPIO1: track 0.00 -> 15.2 mm, vias 0 -> 1
- net /BAT_IN: track 21.7 -> 10.2 mm
- net Net-(U4-VSENSE): track 11.0 -> 0.00 mm
- net /GLOB_GPIO2: track 0.00 -> 9.78 mm, vias 0 -> 1
- net Net-(JP6-B): track 0.00 -> 8.16 mm
- net +3.3V: track 140.2 -> 148.1 mm, vias 20 -> 21
- net +BATT: track 106.0 -> 98.9 mm
- net /LIPO_NTC: track 43.6 -> 46.4 mm
- net Net-(JP6-A): track 0.00 -> 2.09 mm
- net /5V_ENA: track 34.6 -> 36.6 mm
- net /GLOB_~{OFF}: track 125.7 -> 127.6 mm, vias 7 -> 8
- net /I2C_INT: track 88.7 -> 90.6 mm
- net /esp32-c3/TARG_RX: track 18.0 -> 19.9 mm
- net +5V: track 30.0 -> 28.2 mm, vias 1 -> 0
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Other:
- board text added: "BQ_HARDRST"
- board text added: "IO1"
- board text added: "LIPO_BYPASS"
- board text added: "OFF GND 3V3 SCL SDA INT"
- board text added: "USB_CONN"

Commit message: 05/24 order
Parts:
- C43: value 22uF/6.3V -> 2u2
- R18, R29: value 2.2k -> 3k
- moved R25 19.5 mm to (79.0, 92.5)
- moved TP3 2.35 mm to (90.0, 77.0)
Routing:
- net /GLOB_~{OFF}: track 127.6 -> 108.1 mm, vias 8 -> 6
- net /WS2812: track 35.0 -> 32.9 mm
- net /5V_ENA: track 36.6 -> 38.4 mm, vias 1 -> 2
- net /esp32-c3/IO9: track 39.8 -> 40.8 mm
Other:
- board text added: "i2current 05/24 @cb1t"

Commit message: start order
Parts:
- removed C16: 10u, Capacitor_SMD:C_0603_1608Metric
- removed C24, C28: 22uF/6.3V, Capacitor_SMD:C_0603_1608Metric
- removed C7: 100n, Capacitor_SMD:C_0402_1005Metric
- removed D3: 1N5819WS, Diode_SMD:D_SOD-323
- removed J7: Conn_01x05, Connector_PinHeader_1.27mm:PinHeader_1x05_P1.27mm_Vertical
- removed JP2: LIPO_BYPASS, Jumper:SolderJumper-2_P1.3mm_Open_TrianglePad1.0x1.5mm
- removed JP5: USB_CONN, Jumper:SolderJumper-2_P1.3mm_Open_TrianglePad1.0x1.5mm
- removed JP6: 5V_ENA, Jumper:SolderJumper-2_P1.3mm_Open_TrianglePad1.0x1.5mm
- removed L4: FXL0630-6R8-M, easyeda2kicad:IND-SMD_L7.0-W6.6
- removed LED1, LED2, LED3, LED4, LED5: XL-1606UGC, easyeda2kicad:LED-SMD_L1.7-W1.1-R-RD_GREEN
- removed R13: 5.1k/DNP, Resistor_SMD:R_0603_1608Metric_Pad0.98x0.95mm_HandSolder
- removed R15: 10k, Resistor_SMD:R_0402_1005Metric
- removed R17, R30: 6k/0603, Resistor_SMD:R_0603_1608Metric_Pad0.98x0.95mm_HandSolder
- removed R22: 0603/DNP, Resistor_SMD:R_0603_1608Metric_Pad0.98x0.95mm_HandSolder
- removed R26: 3k, Resistor_SMD:R_0402_1005Metric
- removed SW3, SW4: B2, Button_Switch_SMD:SW_SPST_TL3342
- added J4: Conn_01x12_MountingPin, Connector_Molex:Molex_PicoBlade_53261-1271_1x12-1MP_P1.25mm_Horizontal, F.Cu at (73.0, 103.4)
- added R33: 75k, Resistor_SMD:R_0402_1005Metric, F.Cu at (82.5, 80.7)
- added R35: 16k, Resistor_SMD:R_0402_1005Metric, F.Cu at (81.5, 80.7)
- added TP4: TestPoint, TestPoint:TestPoint_Pad_D1.0mm, F.Cu at (91.9, 74.2)
- added U1: SPX3819M5-L-3-3, Package_TO_SOT_SMD:SOT-23-5, F.Cu at (71.8, 78.5)
- added U12: A-SP1102AR6GHC-A01-2C, easyeda2kicad:LED-SMD_4P-L3.0-W1.5_A-SP1102AR6GHC-A01-2C, F.Cu at (49.7, 73.8)
- added U13: A-SP1102AR6GHC-A01-2C, easyeda2kicad:LED-SMD_4P-L3.0-W1.5_A-SP1102AR6GHC-A01-2C, F.Cu at (49.8, 87.9)
- added U6: MT2492, easyeda2kicad:SOT-23-6_L2.9-W1.6-P0.95-LS2.8-BL, F.Cu at (80.5, 77.7)
- C10: value 47p -> 10u; footprint Capacitor_SMD:C_0402_1005Metric -> Capacitor_SMD:C_0603_1608Metric
- C22: value 1n -> 10u; footprint Capacitor_SMD:C_0402_1005Metric -> Capacitor_SMD:C_0603_1608Metric
- C23: value 22uF/6.3V -> 10u
- C3: value 22uF/6.3V -> 22n; footprint Capacitor_SMD:C_0603_1608Metric -> Capacitor_SMD:C_0402_1005Metric
- C8: value 100n -> 22uF/6.3V; footprint Capacitor_SMD:C_0402_1005Metric -> Capacitor_SMD:C_0603_1608Metric
- C9: value 10n -> 22uF/6.3V; footprint Capacitor_SMD:C_0402_1005Metric -> Capacitor_SMD:C_0603_1608Metric
- J1: value ~ -> B4P
- J6: value Conn_01x10 -> Conn_01x05; footprint Connector_Molex:Molex_PicoBlade_53261-1071_1x10-1MP_P1.25mm_Horizontal -> Connector_PinHeader_1.27mm:PinHeader_1x05_P1.27mm_Vertical
- J8: value Conn_01x06 -> PANEL_CONN
- JP4: value USB_CONN -> 3V3_5V; moved to F.Cu
- R1: value 73.2k -> 75k
- R10: value 5.1k/DNP -> 10k; footprint Resistor_SMD:R_0603_1608Metric_Pad0.98x0.95mm_HandSolder -> Resistor_SMD:R_0402_1005Metric
- R11: value 10k -> 100
- R16: value 30k -> 10k
- R20: value 100k -> 75k
- R25: value 6k/0603 -> 3k; footprint Resistor_SMD:R_0603_1608Metric_Pad0.98x0.95mm_HandSolder -> Resistor_SMD:R_0402_1005Metric
- TP1: moved to F.Cu
- TP3: value WS2812_PIN -> TestPoint; footprint TestPoint:TestPoint_THTPad_D1.5mm_Drill0.7mm -> TestPoint:TestPoint_Pad_D1.0mm
- U4: value TPS5430DDA -> FTC252010S4R7MBCA; footprint Package_SO:SOIC-8_3.9x4.9mm_P1.27mm -> easyeda2kicad:IND-SMD_L2.5-W2.0-VLS252012CX-150M
- moved R10 41.6 mm to (84.6, 102.2), turned to 90 degrees
- moved R2 39.5 mm to (83.5, 80.7), turned to -90 degrees
- moved R25 29.8 mm to (57.9, 71.6), turned to 180 degrees
- moved C5 26.8 mm to (62.5, 98.1), turned to 90 degrees
- moved TP2 24.2 mm to (87.8, 74.2)
- moved C1 23.7 mm to (85.6, 102.2), turned to 90 degrees
- moved R9 23.3 mm to (59.9, 86.5), turned to 0 degrees
- moved R16 18.5 mm to (53.8, 71.6), turned to 180 degrees
- moved R12 17.2 mm to (71.6, 82.6), turned to 0 degrees
- moved R6 17.1 mm to (71.6, 84.7)
- moved R5 16.9 mm to (71.6, 83.6), turned to 0 degrees
- moved JP4 16.3 mm to (78.6, 85.2)
- moved J6 13.1 mm to (84.8, 104.7), turned to 90 degrees
- moved R11 12.7 mm to (59.9, 88.5)
- moved R14 11.3 mm to (83.0, 82.2), turned to 180 degrees
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Connections:
- C1 pad 1: /esp32-c3/ESP_EN -> /ESP_EN
- C10 pad 1: GND -> +BATT
- C10 pad 2: Net-(U4-COMP) -> GND
- C11 pad 2: +3.3V -> VDD
- C12 pad 2: +3.3V -> VDD
- C2 pad 1: /esp32-c3/IO9 -> /PWRBRD_BOOT
- C22 pad 1: Net-(C22-Pad1) -> +BATT
- C22 pad 2: Net-(U4-COMP) -> GND
- C23 pad 1: +3.3V -> VDD
- C3 pad 1: +3.3V -> /3V3_L
- C3 pad 2: GND -> Net-(U6-BS)
- C43 pad 1: +3.3V -> VDD
- C44 pad 1: +3.3V -> VDD
- C5 pad 1: +BATT -> +3.3V
- C8 pad 1: /3V3_L -> +3.3V
- C8 pad 2: Net-(U4-BOOT) -> GND
- C9 pad 1: GND -> +3.3V
- C9 pad 2: Net-(U4-SS) -> GND
- J5 pad 10: +3.3V -> +5V
- J5 pad 11: /GLOB_~{OFF} -> /MCU_IO3
- J5 pad 12: /SDA -> /PWRBRD_BOOT
- J5 pad 13: /GLOB_GPIO1 -> GND
- J5 pad 14: /SCL -> /I2C_INT
- J5 pad 15: /GLOB_GPIO2 -> /PWRBRD_TX
- J5 pad 16: GND -> /SDA
- J5 pad 17: GND -> /PWRBRD_RX
- J5 pad 18: Net-(J5-Pin_18) -> /SCL
- J5 pad 19: VBUS -> /GLOB_~{OFF}
- J5 pad 20: Net-(J5-Pin_20) -> +3.3V
- J5 pad 7: VBUS -> /MCU_IO1
- J5 pad 8: /I2C_INT -> /MCU_IO2
- J5 pad 9: +3.3V -> +5V
- J6 pad 1: +VDC -> /ESP_EN
- J6 pad 2: +BATT -> /PWRBRD_BOOT
- J6 pad 4: /I2C_INT -> /PWRBRD_TX
- J6 pad 5: +3.3V -> /PWRBRD_RX
- J8 pad 3: +3.3V -> VDD
- JP4 pad 1: Net-(J5-Pin_20) -> +5V
- JP4 pad 2: /USBIN_P -> +3.3V
- R10 pad 1: GND -> /ESP_EN
- R10 pad 2: /CC1 -> +3.3V
- R11 pad 1: Net-(JP6-B) -> Net-(SW6-A)
- R11 pad 2: +3.3V -> VDD
- R12 pad 2: +3.3V -> VDD
- R14 pad 1: GND -> /5V_ENA
- R14 pad 2: Net-(JP6-B) -> /GLOB_~{OFF}
- R16 pad 1: GND -> /BQ_STAT
- R16 pad 2: Net-(C22-Pad1) -> VDD
- R18 pad 1: /BQ_REGN -> /BQ_STAT
- R2 pad 1: GND -> /3V3_ENA
- R2 pad 2: Net-(LED2-K) -> /GLOB_~{OFF}
- R25 pad 1: /5V_ENA -> GND
- R25 pad 2: /GLOB_~{OFF} -> Net-(R25-Pad2)
- R29 pad 2: GND -> /PWRBRD_STAT
- R5 pad 2: +3.3V -> VDD
- R6 pad 2: +3.3V -> VDD
- R9 pad 1: GND -> Net-(R9-Pad1)
- R9 pad 2: Net-(LED5-K) -> +5V
- TP1 pad 1: Net-(U11-PG) -> /5V_ENA
- TP2 pad 1: /BQ_REGN -> /5V_PG
- TP3 pad 1: /WS2812 -> /3V3_ENA
- U11 pad 4: Net-(U11-PG) -> /5V_PG
- U4 pad 1: Net-(U4-BOOT) -> /3V3_L
- U4 pad 2: +BATT -> +3.3V
- U5 pad 12: +3.3V -> VDD
- U5 pad 13: +3.3V -> VDD
- U5 pad 3: +3.3V -> VDD
- U5 pad 4: +3.3V -> VDD
- U7 pad 11: /esp32-c3/TARG_RX -> /PWRBRD_RX
- U7 pad 12: /esp32-c3/TARG_TX -> /PWRBRD_TX
- U7 pad 15: /GLOB_GPIO2 -> /MCU_IO3
- U7 pad 16: /GLOB_GPIO1 -> /MCU_IO2
- U7 pad 17: /WS2812 -> /MCU_IO1
- U7 pad 18: /esp32-c3/IO0 -> unconnected-(U7-GPIO0/ADC1_CH0/XTAL_32K_P-Pad18)
- U7 pad 2: /esp32-c3/ESP_EN -> /ESP_EN
- U7 pad 4: /esp32-c3/IO5 -> /5V_PG
- U7 pad 5: /esp32-c3/IO6 -> /PWRBRD_STAT
- U7 pad 8: /esp32-c3/IO9 -> /PWRBRD_BOOT
- U8 pad 1: Net-(LED3-K) -> /BQ_STAT
- U8 pad 13: /BQ_REGN -> GND
Routing:
- net +3.3V: track 148.1 -> 27.4 mm, vias 21 -> 11
- net VDD: track 0.00 -> 80.8 mm, vias 0 -> 7
- net +BATT: track 98.9 -> 28.2 mm, vias 25 -> 10
- net /PWRBRD_BOOT: track 0.00 -> 60.1 mm, vias 0 -> 7
- net /5V_PG: track 0.00 -> 58.9 mm, vias 0 -> 7
- net +5V: track 28.2 -> 81.9 mm, vias 0 -> 10
- net /esp32-c3/ESP_EN: track 50.5 -> 0.00 mm, vias 3 -> 0
- net /esp32-c3/IO9: track 40.8 -> 0.00 mm, vias 7 -> 0
- net VBUS: track 91.4 -> 50.9 mm, vias 10 -> 8
- net /PWRBRD_TX: track 0.00 -> 40.3 mm, vias 0 -> 2
- net +VDC: track 68.4 -> 28.1 mm, vias 15 -> 6
- net /GLOB_~{OFF}: track 108.1 -> 143.7 mm, vias 6 -> 3
- net /PWRBRD_RX: track 0.00 -> 33.2 mm, vias 0 -> 2
- net /WS2812: track 32.9 -> 0.00 mm, vias 2 -> 0
- net /MCU_IO2: track 0.00 -> 28.2 mm, vias 0 -> 1
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- added copper zone on B.Cu, net +5V
- removed copper zone on F.Cu, net /BQ_REGN
Other:
- outline, holes or cut-outs redrawn
- board text added: "3K->1S 6K->2S 10.5K->3S 17.4K->4S"
- board text added: "3V3"
- board text added: "5V0"
- board text added: "BAT"
- board text added: "CHG"
- board text added: "GND"
- board text added: "IO1|IO2 5V0|5V0 IO3|IO9 GND|INT BTX|SDA BRX|SCL OFF|3V3"
- board text added: "PWRMUX"
- board text added: "VDC"
- board text added: "VDD"
- board text added: "i2current 08/24 @clue.lamp @cb1t @elektrojakub"
- board text removed: "3V3-5V"
- board text removed: "BOOT"
- board text removed: "CHG 1-4S"
- board text removed: "IO1"
- board text removed: "RST"
- board text removed: "i2current 05/24 @cb1t"
- board text removed: "pwr mux"
