File: i2current.kicad_pcb (KiCad board)
At the start: 2 copper layers, 50 x 64 mm, 109 parts, among them CN1 JL15EDGA-38106G01, J1 B4P, J10 QWIIC, J11 QWIIC, J2 USB_C_Receptacle_USB2.0, J3 CONN_BATT, J4 Conn_01x12_MountingPin, J5 EXT_IFACE, J6 Conn_01x05, J8 PANEL_CONN, J9 Conn_01x06, Q1 AO3400A, Q4 AO3400A, Q5 AO3400A, Q6 AO3400A, Q8 AO3400A, SW6 SW_SPDT, U1 SPX3819M5-L-3-3, U10 SMTSO3030CTJ, U11 TPS56637RPAR, U12 A-SP1102AR6GHC-A01-2C, U13 A-SP1102AR6GHC-A01-2C, U2 SMTSO3030CTJ, U3 SMTSO3030CTJ, U4 FTC252010S4R7MBCA, U5 FUSB302B01MPX, U6 MT2492, U7 ESP32-C3-WROOM-02, U8 BQ25792RQMR, U9 SMTSO3030CTJ

Commit message: checkpoint for next rev
Parts:
- removed J10, J11: QWIIC, Connector_JST:JST_SH_SM04B-SRSS-TB_1x04-1MP_P1.00mm_Horizontal
- removed J6: Conn_01x05, Connector_PinHeader_1.27mm:PinHeader_1x05_P1.27mm_Vertical
- removed J8: PANEL_CONN, Connector_PinHeader_2.54mm:PinHeader_1x06_P2.54mm_Vertical
- removed J9: Conn_01x06, Connector_JST:JST_PH_S6B-PH-K_1x06_P2.00mm_Horizontal
- removed JP4: 3V3_5V, Jumper:SolderJumper-2_P1.3mm_Open_TrianglePad1.0x1.5mm
- removed Q4, Q5, Q8: AO3400A, Package_TO_SOT_SMD:SOT-23
- removed R29: 3k, Resistor_SMD:R_0402_1005Metric
- removed TP1, TP3, TP4: TestPoint, TestPoint:TestPoint_Pad_D1.0mm
- removed U13: A-SP1102AR6GHC-A01-2C, easyeda2kicad:LED-SMD_4P-L3.0-W1.5_A-SP1102AR6GHC-A01-2C
- added C16: 22n, Capacitor_SMD:C_0402_1005Metric, F.Cu at (74.6, 60.4)
- added C24: 10u, Capacitor_SMD:C_0603_1608Metric, F.Cu at (25.6, 99.3)
- added C28: 10u, Capacitor_SMD:C_0603_1608Metric, F.Cu at (28.1, 99.3)
- added C45: 100n, Capacitor_SMD:C_0402_1005Metric, F.Cu at (30.7, 95.9)
- added C46: 100n, Capacitor_SMD:C_0402_1005Metric, F.Cu at (72.3, 80.5)
- added C47: 10u, Capacitor_SMD:C_0603_1608Metric, F.Cu at (30.6, 99.3)
- added C7: 100u/6.3/tant, Capacitor_THT:CP_Radial_D8.0mm_P5.00mm, B.Cu at (87.8, 53.0)
- added D1: LED, LED_SMD:LED_0805_2012Metric, F.Cu at (94.5, 74.3)
- added D3: LED, LED_SMD:LED_0805_2012Metric, F.Cu at (49.4, 73.7)
- added D4: LED, LED_SMD:LED_0805_2012Metric, F.Cu at (49.2, 87.8)
- added JP2: VBUS_VPWR, Jumper:SolderJumper-2_P1.3mm_Open_TrianglePad1.0x1.5mm, F.Cu at (82.3, 83.0)
- added JP5: VSYS_VBUS, Jumper:SolderJumper-2_P1.3mm_Open_TrianglePad1.0x1.5mm, F.Cu at (111.4, 84.7)
- added Q2: AON7544, easyeda2kicad:DFN-8_L3.3-W3.3-P0.65-BL-2, F.Cu at (61.3, 73.3)
- added Q3: AON7544, easyeda2kicad:DFN-8_L3.3-W3.3-P0.65-BL-2, F.Cu at (66.0, 73.3)
- added R13: 16k, Resistor_SMD:R_0603_1608Metric, F.Cu at (81.3, 73.5)
- added R15: 100, Resistor_SMD:R_0402_1005Metric, F.Cu at (65.7, 76.0)
- added R17: 100, Resistor_SMD:R_0402_1005Metric, F.Cu at (65.7, 77.1)
- added R22: 3k, Resistor_SMD:R_0402_1005Metric, F.Cu at (70.5, 80.9)
- added R26: 10k, Resistor_SMD:R_0402_1005Metric, F.Cu at (76.5, 78.8)
- C1, C2: value 100n -> 22uF/25V; footprint Capacitor_SMD:C_0402_1005Metric -> Capacitor_SMD:C_1206_3216Metric
- C15: value 22uF/6.3V -> 100u/6.3/tant; footprint Capacitor_SMD:C_0603_1608Metric -> Capacitor_Tantalum_SMD:CP_EIA-3528-21_Kemet-B
- C26, C42, C6: value 10u -> 100n; footprint Capacitor_SMD:C_0603_1608Metric -> Capacitor_SMD:C_0402_1005Metric
- C4: value 22uF/6.3V -> 200p; footprint Capacitor_SMD:C_0603_1608Metric -> Capacitor_SMD:C_0402_1005Metric
- C41: value 22uF/6.3V -> 22uF/25V; footprint Capacitor_SMD:C_0603_1608Metric -> Capacitor_SMD:C_1206_3216Metric
- C43: value 2u2 -> 100n; footprint Capacitor_SMD:C_0603_1608Metric -> Capacitor_SMD:C_0402_1005Metric
- Q1, Q6: value AO3400A -> AON7544; footprint Package_TO_SOT_SMD:SOT-23 -> easyeda2kicad:DFN-8_L3.3-W3.3-P0.65-BL-2
- R1, R20, R21, R3, R33, R35, R7, R8: footprint Resistor_SMD:R_0402_1005Metric -> Resistor_SMD:R_0603_1608Metric
- R10: value 10k -> 2
- R18, R25: value 3k -> 10k
- R27, R28: value 300/0603 -> 3k; footprint Resistor_SMD:R_0603_1608Metric_Pad0.98x0.95mm_HandSolder -> Resistor_SMD:R_0402_1005Metric
- R9: value 10k -> 16k; footprint Resistor_SMD:R_0402_1005Metric -> Resistor_SMD:R_0603_1608Metric
- TP2: moved to B.Cu
- U12: value A-SP1102AR6GHC-A01-2C -> PY32F002AW15U6TR; footprint easyeda2kicad:LED-SMD_4P-L3.0-W1.5_A-SP1102AR6GHC-A01-2C -> Package_DFN_QFN:TQFN-16-1EP_3x3mm_P0.5mm_EP1.6x1.6mm
- U7: value ESP32-C3-WROOM-02 -> JLC_OLED; footprint Espressif:ESP32-C3-WROOM-02 -> Critbit_lib:OLED-042-JLC
- moved C6 63.2 mm to (22.8, 95.9), turned to 90 degrees
- moved C42 62.2 mm to (26.7, 95.9), turned to 90 degrees
- moved C26 61.0 mm to (24.8, 95.9), turned to 90 degrees
- moved C5 39.4 mm to (23.1, 99.3)
- moved C1 39.3 mm to (78.2, 63.6)
- moved C43 37.1 mm to (28.7, 95.9), turned to 90 degrees
- moved C2 33.8 mm to (78.0, 69.5), turned to -90 degrees
- moved R9 33.2 mm to (90.7, 74.1), turned to 180 degrees
- moved R33 31.2 mm to (90.0, 111.0)
- moved JP1 30.3 mm to (39.8, 65.2), turned to 90 degrees
- moved C3 29.5 mm to (87.7, 108.4)
- moved C8 29.5 mm to (87.6, 109.7)
- moved C9 29.5 mm to (87.5, 111.2)
- moved R35 29.5 mm to (90.0, 109.0)
- moved U4 29.5 mm to (85.7, 105.9)
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Connections:
- net /3V3_L renamed /VMCU_L
- C1 pad 1: /ESP_EN -> SYS
- C10 pad 1: +BATT -> SYS
- C11 pad 2: VDD -> 3V3_SYS
- C12 pad 2: VDD -> 3V3_SYS
- C15 pad 1: +5V -> VPWR
- C2 pad 1: /PWRBRD_BOOT -> SYS
- C22 pad 1: +BATT -> SYS
- C23 pad 1: VDD -> 3V3_SYS
- C26 pad 1: +BATT -> GND
- C26 pad 2: GND -> VMCU
- C27 pad 2: +BATT -> SYS
- C29 pad 2: GND -> +VDC
- C30 pad 2: GND -> VBUS
- C31 pad 1: +BATT -> SYS
- C32 pad 1: +BATT -> SYS
- C36 pad 2: +BATT -> SYS
- C37 pad 1: +BATT -> SYS
- C4 pad 1: +5V -> Net-(C4-Pad1)
- C4 pad 2: GND -> Net-(U11-FB)
- C41 pad 1: +5V -> VPWR
- C42 pad 1: /BAT_IN -> GND
- C42 pad 2: GND -> Net-(U7-VCC)
- C43 pad 1: VDD -> Net-(U7-C2P)
- C43 pad 2: GND -> Net-(U7-C2N)
- C44 pad 1: VDD -> 3V3_SYS
- C5 pad 1: +3.3V -> VMCU
- C6 pad 1: +BATT -> GND
- C6 pad 2: GND -> 3V3_SYS
- C8 pad 1: +3.3V -> VMCU
- C9 pad 1: +3.3V -> VMCU
- CN1 pad 1: /BAT_IN -> BAT
- CN1 pad 4: +BATT -> SYS
- J1 pad 5V: +5V -> VPWR
- J3 pad 1: /BAT_IN -> BAT
- J4 pad 12: +5V -> VMCU
- J5 pad 10: +5V -> VPWR
- J5 pad 11: /MCU_IO3 -> /PY32_SWD
- J5 pad 20: +3.3V -> VMCU
- J5 pad 3: +BATT -> SYS
- J5 pad 4: +BATT -> SYS
- J5 pad 7: /MCU_IO1 -> /PY32_SWC
- J5 pad 8: /MCU_IO2 -> /PY32_nRST
- J5 pad 9: +5V -> VPWR
- L1 pad 2: +5V -> VPWR
- Q1 pad 1: Net-(D7-K) -> Net-(D6-A)
- Q1 pad 2: Net-(D7-A) -> Net-(D6-A)
- Q1 pad 3: VBUS_PIN -> Net-(D6-A)
- Q6 pad 1: Net-(Q6-G) -> Net-(D6-A)
- Q6 pad 2: BAT -> Net-(D6-A)
- Q6 pad 3: /BAT_IN -> Net-(D6-A)
- R1 pad 2: +5V -> VPWR
- R10 pad 1: /ESP_EN -> GND
- R10 pad 2: +3.3V -> /BQ_nCE
- R11 pad 2: VDD -> 3V3_SYS
- R12 pad 2: VDD -> 3V3_SYS
- R16 pad 2: VDD -> 3V3_SYS
- R18 pad 2: Net-(R18-Pad2) -> Net-(D3-K)
- R23 pad 2: +VDC -> GND
- R24 pad 2: VBUS -> GND
- R25 pad 2: Net-(R25-Pad2) -> Net-(D4-K)
- R27 pad 1: Net-(U8-ACDRV2) -> GND
- R27 pad 2: Net-(D6-K) -> /PY32_ADC
- R28 pad 1: Net-(U8-ACDRV1) -> /PY32_ADC
- R28 pad 2: Net-(D7-K) -> VPWR
- R33 pad 2: +3.3V -> VMCU
- R4 pad 2: /BAT_IN -> BAT
- R5 pad 2: VDD -> 3V3_SYS
- R6 pad 2: VDD -> 3V3_SYS
- R9 pad 2: +5V -> VPWR
- U1 pad 1: +BATT -> SYS
- U1 pad 3: +BATT -> SYS
- U1 pad 5: VDD -> 3V3_SYS
- U11 pad 8: +BATT -> SYS
- U12 pad 1: VDD -> /3V3_ENA
- U12 pad 2: /GLOB_~{OFF} -> /5V_ENA
- U12 pad 3: Net-(R25-Pad2) -> /PY32_SWD
- U12 pad 4: Net-(R18-Pad2) -> /PY32_SWC
- U4 pad 2: +3.3V -> VMCU
- U5 pad 12: VDD -> 3V3_SYS
- U5 pad 13: VDD -> 3V3_SYS
- U5 pad 3: VDD -> 3V3_SYS
- U5 pad 4: VDD -> 3V3_SYS
- U6 pad 5: +BATT -> SYS
- U7 pad 1: +3.3V -> Net-(U7-C2P)
- U7 pad 10: /5V_ENA -> /OLED_RST
- U7 pad 11: /PWRBRD_RX -> GND
- U7 pad 12: /PWRBRD_TX -> /SCL
- U7 pad 13: /USBIN_M -> /SDA
- U7 pad 14: /USBIN_P -> /SDA
- U7 pad 15: /MCU_IO3 -> Net-(U7-VCOMH)
- U7 pad 16: /MCU_IO2 -> Net-(U7-VCC)
- U7 pad 2: /ESP_EN -> Net-(U7-C2N)
- U7 pad 3: /I2C_INT -> Net-(U7-C1P)
- U7 pad 4: /5V_PG -> Net-(U7-C1N)
- U7 pad 5: /PWRBRD_STAT -> VMCU
- U7 pad 6: /SCL -> GND
- U7 pad 7: /SDA -> 3V3_SYS
- U7 pad 8: /PWRBRD_BOOT -> +3.3V
- U8 pad 13: GND -> /BQ_nCE
- U8 pad 24: Net-(Q6-G) -> Net-(U8-SDRV)
- U8 pad 25: +BATT -> SYS
Routing:
- net 3V3_SYS: track 0.00 -> 86.4 mm, vias 0 -> 8
- net +5V: track 81.9 -> 0.00 mm, vias 10 -> 0
- net VDD: track 80.8 -> 0.00 mm, vias 7 -> 0
- net /5V_PG: track 58.9 -> 0.64 mm, vias 7 -> 1
- net GND: track 155.7 -> 102.9 mm, vias 60 -> 47
- net VPWR: track 0.00 -> 32.3 mm, vias 0 -> 8
- net /PY32_nRST: track 0.00 -> 29.3 mm
- net /MCU_IO2: track 28.2 -> 0.00 mm, vias 1 -> 0
- net +BATT: track 28.2 -> 0.00 mm, vias 10 -> 0
- net /3V3_ENA: track 9.64 -> 37.4 mm
- net +3.3V: track 27.4 -> 0.00 mm, vias 11 -> 0
- net /MCU_IO1: track 27.2 -> 0.00 mm, vias 1 -> 0
- net /PY32_SWD: track 0.00 -> 26.3 mm
- net /ESP_EN: track 25.0 -> 0.00 mm, vias 1 -> 0
- net SYS: track 0.00 -> 24.0 mm, vias 0 -> 17
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- added copper zone on B.Cu, net SYS
- added copper zone on F.Cu, net SYS
- added copper zone on B.Cu, net VMCU
- added copper zone on F.Cu, net VMCU
- added copper zone on B.Cu, net VPWR
- added copper zone on F.Cu, net VPWR
- removed copper zone on B.Cu, net +3.3V
- removed copper zone on F.Cu, net +3.3V
- removed copper zone on B.Cu, net +5V
- removed copper zone on F.Cu, net +5V
- removed copper zone on B.Cu, net +BATT
- removed copper zone on F.Cu, net +BATT
- removed copper zone on B.Cu, net +VDC
- removed copper zone on F.Cu, net /BAT_IN
Other:
- outline, holes or cut-outs redrawn
- board text added: "NTC"
- board text added: "OFF"
- board text added: "PD"
- board text added: "PWR MUX"
- board text added: "SYS"
- board text added: "VIN"
- board text removed: "OFF GND 3V3 SCL SDA INT"
- board text removed: "PWRMUX"
- board text removed: "USBC-PD"

Commit message: finish DRC
Parts:
- removed JP1: HARDRST, Jumper:SolderJumper-2_P1.3mm_Open_TrianglePad1.0x1.5mm
- removed JP2: VBUS_VPWR, Jumper:SolderJumper-2_P1.3mm_Open_TrianglePad1.0x1.5mm
- removed JP5: VSYS_VBUS, Jumper:SolderJumper-2_P1.3mm_Open_TrianglePad1.0x1.5mm
- removed L3: FXL0420-1R0-M, easyeda2kicad:IND-SMD_L4.4-W4.2
- added D2: LED, LED_SMD:LED_0805_2012Metric, F.Cu at (96.0, 103.7)
- added L2: SPM6530T-1R0M120, easyeda2kicad:IND-SMD_L7.1-W6.5-P5.60, F.Cu at (70.0, 59.6)
- added R29: 0R/1206, Resistor_SMD:R_1206_3216Metric, F.Cu at (78.6, 82.2)
- added R30: 0R/1206, Resistor_SMD:R_1206_3216Metric, F.Cu at (82.0, 83.3)
- added R32: 10k, Resistor_SMD:R_0402_1005Metric, F.Cu at (92.9, 103.8)
- added TP1: TestPoint, TestPoint:TestPoint_Pad_D1.0mm, F.Cu at (70.6, 72.4)
- added U13: USBLC6-4SC6, Package_TO_SOT_SMD:SOT-23-6, F.Cu at (53.5, 88.4)
- moved C6 56.6 mm to (79.4, 94.3), turned to 180 degrees
- moved C5 56.1 mm to (78.7, 92.3)
- moved C24 55.5 mm to (80.2, 89.3), turned to -90 degrees
- moved C26 54.6 mm to (79.4, 95.3), turned to 180 degrees
- moved C42 53.4 mm to (79.4, 87.3), turned to 0 degrees
- moved C28 51.6 mm to (78.7, 89.3), turned to -90 degrees
- moved C43 50.7 mm to (79.4, 97.4), turned to 180 degrees
- moved C47 50.1 mm to (80.2, 92.3)
- moved C45 48.7 mm to (79.4, 96.3), turned to 180 degrees
- moved R9 21.3 mm to (90.4, 52.8), turned to -90 degrees
- moved D1 18.5 mm to (90.8, 56.1), turned to -90 degrees
- moved U7 5.92 mm to (79.4, 93.0)
- moved R31 4.15 mm to (78.6, 58.9)
- moved R5 3.32 mm to (71.3, 87.8), turned to -90 degrees
- moved C9 2.47 mm to (85.2, 110.5), turned to -90 degrees
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Connections:
- net Net-(D6-A) renamed /AC2_FETS
- net Net-(D7-A) renamed /AC1_FETS
- D1 pad 1: GND -> Net-(D1-K)
- D1 pad 2: Net-(D1-A) -> VPWR
- R9 pad 1: Net-(D1-A) -> GND
- R9 pad 2: VPWR -> Net-(D1-K)
- U7 pad 8: +3.3V -> 3V3_SYS
Routing:
- net SYS: track 24.0 -> 72.0 mm
- net GND: track 102.9 -> 149.0 mm, vias 47 -> 68
- net /OLED_RST: track 0.00 -> 22.9 mm, vias 0 -> 3
- net VMCU: track 5.36 -> 26.1 mm, vias 4 -> 9
- net /GLOB_~{OFF}: track 133.9 -> 153.2 mm, vias 8 -> 11
- net Net-(D6-K): track 0.00 -> 11.6 mm
- net 3V3_SYS: track 86.4 -> 97.9 mm, vias 8 -> 12
- net /USBIN_M: track 41.3 -> 52.6 mm
- net /CC1: track 15.2 -> 26.4 mm
- net Net-(U8-~{QON}): track 12.0 -> 2.58 mm
- net /USBIN_P: track 41.7 -> 50.8 mm
- net /PWRBRD_BOOT: track 51.1 -> 59.7 mm
- net Net-(D7-K): track 2.02 -> 9.49 mm
- net /BQ_SW1: track 7.60 -> 14.2 mm, vias 5 -> 7
- net /CC2: track 14.4 -> 20.2 mm, vias 0 -> 2
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- added copper zone on F.Cu, net /AC1_FETS
- added copper zone on F.Cu, net /AC2_FETS
Other:
- outline, holes or cut-outs redrawn
- board text added: "1"
- board text added: "16"
- board text added: "@cb1t + @elektrojakub"
- board text added: "CTRL"
- board text added: "Rprog"
- board text added: "Rprog: 3K->1S 6K->2S 10.5K->3S 17.4K->4S"
- board text added: "SW"
- board text added: "SWC|RST"
- board text added: "SWD|BOT GND|INT BTX|SDA BRX|SCL OFF|Vmcu"
- board text added: "USB->5V"
- board text added: "USB->SYS"
- board text added: "Vmcu"
- board text added: "Vpwr"
- board text added: "Vsys"
- board text added: "i2current 01/25 for @clue.lamp"
- board text removed: "3K->1S 6K->2S 10.5K->3S 17.4K->4S"
- board text removed: "3V3"
- board text removed: "5V"
- board text removed: "5V0"
- board text removed: "IO1|IO2 5V0|5V0 IO3|IO9 GND|INT BTX|SDA BRX|SCL OFF|3V3"
- board text removed: "USB_CONN"
- board text removed: "i2current 08/24 @clue.lamp @cb1t @elektrojakub"

Commit message: before parts
Parts:
- removed U10, U2, U3, U9: SMTSO3030CTJ, easyeda2kicad:SMD_BD5.6-D4.1
- added C48: 100n, Capacitor_SMD:C_0402_1005Metric, F.Cu at (59.2, 71.0)
- added C49: 100n, Capacitor_SMD:C_0402_1005Metric, F.Cu at (56.0, 76.6)
- added D10: SMF24CA, easyeda2kicad:SOD-123FL_L2.7-W1.8-LS3.8-BI, F.Cu at (78.2, 58.6)
- added D5: 1N5819WS, Diode_SMD:D_SOD-323, F.Cu at (60.5, 57.1)
- added D8: SMF24CA, easyeda2kicad:SOD-123FL_L2.7-W1.8-LS3.8-BI, F.Cu at (60.2, 83.6)
- added D9: SMF24CA, easyeda2kicad:SOD-123FL_L2.7-W1.8-LS3.8-BI, F.Cu at (54.8, 56.4)
- added H1: M3_HOLE, MountingHole:MountingHole_3.2mm_M3_DIN965_Pad, F.Cu at (51.5, 52.0)
- added H2: M3_HOLE, MountingHole:MountingHole_3.2mm_M3_DIN965_Pad, F.Cu at (94.5, 52.0)
- added H3: M3_HOLE, MountingHole:MountingHole_3.2mm_M3_DIN965_Pad, F.Cu at (51.5, 109.0)
- added H4: M3_HOLE, MountingHole:MountingHole_3.2mm_M3_DIN965_Pad, F.Cu at (94.5, 109.0)
- added R34: 5.1k_0603, Resistor_SMD:R_0603_1608Metric, F.Cu at (51.4, 88.8)
- added R36: 5.1k_0603, Resistor_SMD:R_0603_1608Metric, F.Cu at (57.0, 86.2)
- added TP10: TestPoint, TestPoint:TestPoint_Pad_D1.0mm, B.Cu at (95.8, 92.8)
- added TP11: TestPoint, TestPoint:TestPoint_Pad_D1.0mm, B.Cu at (85.0, 83.5)
- added TP12: TestPoint, TestPoint:TestPoint_Pad_D1.0mm, B.Cu at (87.5, 85.0)
- added TP13: TestPoint, TestPoint:TestPoint_Pad_D1.0mm, B.Cu at (87.5, 90.2)
- added TP14: TestPoint, TestPoint:TestPoint_Pad_D1.0mm, B.Cu at (87.5, 92.7)
- added TP15: TestPoint, TestPoint:TestPoint_Pad_D2.0mm, B.Cu at (53.5, 57.0)
- added TP16: TestPoint, TestPoint:TestPoint_Pad_D2.0mm, B.Cu at (91.8, 102.0)
- added TP3: TestPoint, TestPoint:TestPoint_Pad_D2.0mm, B.Cu at (56.5, 57.0)
- added TP4: TestPoint, TestPoint:TestPoint_Pad_D2.0mm, B.Cu at (89.5, 104.0)
- added TP5: TestPoint, TestPoint:TestPoint_Pad_D1.0mm, B.Cu at (51.8, 79.0)
- added TP6: TestPoint, TestPoint:TestPoint_Pad_D1.0mm, B.Cu at (51.8, 82.0)
- added TP7: TestPoint, TestPoint:TestPoint_Pad_D1.0mm, B.Cu at (53.8, 80.5)
- added TP8: TestPoint, TestPoint:TestPoint_Pad_D1.0mm, B.Cu at (95.8, 95.2)
- added TP9: TestPoint, TestPoint:TestPoint_Pad_D1.0mm, B.Cu at (95.8, 97.8)
- R13, R9: value 16k -> 20k_0603
- R29, R30: value 0R/1206 -> 0R_1206
- R3: value 10k -> 10k_0603
- R31: value 10k/0603/DNP -> 10k_0603
- R32: value 10k -> 20k_0603; footprint Resistor_SMD:R_0402_1005Metric -> Resistor_SMD:R_0603_1608Metric
- R35: value 16k -> 10k_0603
- R7: value 5k -> 5.6k
- R8: value 30k -> 33k
- moved R9 21.2 mm to (91.0, 74.0), turned to 0 degrees
- moved D1 18.5 mm to (94.3, 74.2), turned to 0 degrees
- moved R31 13.0 mm to (91.5, 57.1), turned to 180 degrees
- moved R11 1.40 mm to (53.8, 90.8)
- moved R25 1.02 mm to (51.8, 90.8), turned to 180 degrees
- moved U13 0.93 mm to (54.4, 88.5)
- moved R32 0.15 mm to (92.8, 103.8)
Connections:
- C16 pad 2: Net-(U8-SDRV) -> BAT
- U8 pad 24: Net-(U8-SDRV) -> BAT
Routing:
- net GND: track 149.0 -> 160.8 mm, vias 68 -> 74
- net Net-(U8-SDRV): track 6.22 -> 0.00 mm, vias 2 -> 0
- net BAT: track 10.4 -> 16.6 mm, vias 7 -> 9
- net Net-(D5-K): track 0.00 -> 5.96 mm, vias 0 -> 1
- net /LIPO_NTC: track 52.1 -> 56.7 mm
- net VBUS: track 56.3 -> 52.8 mm, vias 9 -> 8
- net 3V3_SYS: track 97.9 -> 94.8 mm
- net /CC1: track 26.4 -> 28.9 mm
- net /CC2: track 20.2 -> 22.5 mm, vias 2 -> 3
- net /GLOB_~{OFF}: track 153.2 -> 151.6 mm
- net /SCL: track 100.0 -> 100.7 mm
- net /I2C_INT: track 102.9 -> 103.5 mm
- net Net-(SW6-A): track 6.74 -> 6.18 mm
Other:
- board text added: "CC1"
- board text added: "CC2"
- board text added: "CPwr"
- board text added: "INT"
- board text added: "SCL"
- board text added: "SDA"
- board text added: "SWC"
- board text added: "SWD"
- board text added: "Ts"
- board text added: "VIN_PROT"
- board text added: "nRST"
- board text removed: "BQ_HARDRST"
- board text removed: "LIPO_BYPASS"

Commit message: really before order really
Parts:
- removed JP3: VBUS_DC, Jumper:SolderJumper-2_P1.3mm_Open_TrianglePad1.0x1.5mm
- added D11: PSM712-LF-T7, easyeda2kicad:SOT-23-3_L3.0-W1.7-P0.95-LS2.9-BR, F.Cu at (62.7, 81.7)
- added D12: LED, LED_SMD:LED_0603_1608Metric, F.Cu at (64.3, 85.2)
- added D13: LED, LED_SMD:LED_0603_1608Metric, F.Cu at (70.8, 82.5)
- added R37: 0R_0805, Resistor_SMD:R_0805_2012Metric, F.Cu at (57.6, 78.1)
- added R38: 75k, Resistor_SMD:R_0603_1608Metric, F.Cu at (56.5, 57.1)
- added R39: 75k, Resistor_SMD:R_0603_1608Metric, F.Cu at (66.7, 84.5)
- added R40: 10k, Resistor_SMD:R_0402_1005Metric, F.Cu at (70.0, 80.5)
- C10, C17, C18, C22, C23, C24, C28, C31, C32, C33, C34, C37, C39, C40, C47, C5: value 10u -> 10u/25V
- C13, C14, C4: value 200p -> 220p
- C29, C30: value 2u2 -> 1u/25V
- C7: value 100u/6.3/tant -> 100u/tht
- D1, D2, D3, D4: footprint LED_SMD:LED_0805_2012Metric -> LED_SMD:LED_0603_1608Metric
- D6: value 1N5819WS -> PSM712-LF-T7; footprint Diode_SMD:D_SOD-323 -> easyeda2kicad:SOT-23-3_L3.0-W1.7-P0.95-LS2.9-BR
- D7: value 1N5819WS -> LED; footprint Diode_SMD:D_SOD-323 -> LED_SMD:LED_0603_1608Metric
- R10, R23, R24: footprint Resistor_SMD:R_0402_1005Metric -> Resistor_SMD:R_0603_1608Metric
- R29, R30: value 0R_1206 -> 0R_0805; footprint Resistor_SMD:R_1206_3216Metric -> Resistor_SMD:R_0805_2012Metric
- R31: footprint Resistor_SMD:R_0603_1608Metric_Pad0.98x0.95mm_HandSolder -> Resistor_SMD:R_0603_1608Metric
- moved D7 18.9 mm to (53.4, 57.1), turned to 0 degrees
- moved D9 16.7 mm to (60.8, 71.9), turned to 180 degrees
- moved TP5 9.53 mm to (51.0, 88.5)
- moved TP6 9.02 mm to (58.0, 88.5)
- moved C49 8.14 mm to (57.5, 84.6), turned to 90 degrees
- moved TP7 8.04 mm to (54.5, 88.5)
- moved D6 5.99 mm to (62.8, 74.6)
- moved R11 4.22 mm to (55.4, 94.7), turned to -90 degrees
- moved R22 3.32 mm to (73.8, 80.9), turned to 90 degrees
- moved R29 3.18 mm to (81.7, 81.3), turned to 0 degrees
- moved R36 3.10 mm to (54.0, 87.0)
- moved C44 3.02 mm to (54.4, 70.3), turned to 0 degrees
- moved C11 2.89 mm to (51.9, 73.5), turned to 90 degrees
- moved C29 2.83 mm to (60.0, 77.4)
- moved C30 2.69 mm to (60.0, 79.0)
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Connections:
- D6 pad 1: Net-(D6-K) -> Net-(Q2-G)
- D6 pad 2: /AC2_FETS -> Net-(Q2-G)
- D7 pad 1: Net-(D7-K) -> GND
- D7 pad 2: /AC1_FETS -> Net-(D7-A)
- Q1 pad 4: Net-(D6-K) -> Net-(Q1-G)
- Q2 pad 4: Net-(D7-K) -> Net-(Q2-G)
- Q3 pad 4: Net-(D7-K) -> Net-(Q2-G)
- Q6 pad 4: Net-(D6-K) -> Net-(Q1-G)
- R15 pad 1: Net-(D7-K) -> Net-(Q2-G)
- R17 pad 1: Net-(D6-K) -> Net-(Q1-G)
Routing:
- net /GLOB_~{OFF}: track 151.6 -> 134.7 mm, vias 11 -> 10
- net GND: track 160.8 -> 173.8 mm, vias 74 -> 80
- net Net-(Q1-G): track 0.00 -> 12.5 mm
- net Net-(D6-K): track 11.6 -> 0.00 mm
- net Net-(Q2-G): track 0.00 -> 9.70 mm
- net Net-(D7-K): track 9.49 -> 0.00 mm
- net Net-(U12-PA6): track 1.98 -> 9.00 mm
- net /BQ_STAT: track 34.3 -> 27.4 mm, vias 4 -> 2
- net /SDA: track 103.6 -> 109.2 mm
- net SYS: track 72.0 -> 66.9 mm
- net /SCL: track 100.7 -> 105.0 mm
- net Net-(U8-ACDRV1): track 9.61 -> 13.4 mm
- net /I2C_INT: track 103.5 -> 106.9 mm
- net /CC2: track 22.5 -> 25.5 mm
- net Net-(D13-K): track 0.00 -> 2.07 mm
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- added copper zone on F.Cu, net 3V3_SYS
Other:
- board text added: "3V3"
- board text added: "ON"
- board text added: "PWRMUX"
- board text added: "Vin"
- board text added: "Vusb"
- board text added: "pwr"
- board text added: "sys"
- board text added: "usb"
- board text removed: "PWR MUX"
- board text removed: "SW"
- board text removed: "USB->5V"
- board text removed: "USB->SYS"
- board text removed: "VDD"

Commit message: PCB next rev checkpoint
Parts:
- removed CN1: JL15EDGA-38106G01, easyeda2kicad:CONN-TH_6P-P3.81_JILN_JL15EDGA-38106G01
- removed J3: CONN_BATT, Connector_JST:JST_PH_S3B-PH-K_1x03_P2.00mm_Horizontal
- removed R29, R30: 0R_0805, Resistor_SMD:R_0805_2012Metric
- added C50: 22uF/25V, Capacitor_SMD:C_1206_3216Metric, F.Cu at (91.6, 62.8)
- added C51: 10u/25V, Capacitor_SMD:C_0603_1608Metric, F.Cu at (86.8, 72.3)
- added CN2: JL15EDGA-38108G01, easyeda2kicad:CONN-TH_8P-P3.81_JILN_JL15EDGA-38108G01, F.Cu at (73.0, 51.6)
- added JP1: 1S, Jumper:SolderJumper-2_P1.3mm_Open_TrianglePad1.0x1.5mm, F.Cu at (81.1, 70.0)
- added JP2: 2S, Jumper:SolderJumper-2_P1.3mm_Open_TrianglePad1.0x1.5mm, F.Cu at (81.1, 72.6)
- added R41: 3k/0603, Resistor_SMD:R_0603_1608Metric, F.Cu at (77.9, 70.2)
- added R42: 3k/0603, Resistor_SMD:R_0603_1608Metric, F.Cu at (77.9, 68.7)
- added R43: 3k/0603, Resistor_SMD:R_0603_1608Metric, F.Cu at (77.9, 71.7)
- added R44: 3k/0603, Resistor_SMD:R_0603_1608Metric, F.Cu at (77.9, 73.2)
- added R45: 100, Resistor_SMD:R_0402_1005Metric, F.Cu at (68.2, 128.0)
- added REF**: PinHeader_1x03_P2.54mm_Horizontal, Connector_PinHeader_2.54mm:PinHeader_1x03_P2.54mm_Horizontal, F.Cu at (97.0, 69.6)
- added TP17: TestPoint, Critbit_lib:Nano_testpad_0.5x1.0mm, F.Cu at (70.6, 71.7)
- added TP18: TestPoint, Critbit_lib:Nano_testpad_0.5x1.0mm, B.Cu at (64.3, 62.4)
- added TP19: TestPoint, Critbit_lib:Nano_testpad_0.5x1.0mm, F.Cu at (64.3, 62.4)
- added TP20: TestPoint, TestPoint:TestPoint_Pad_D1.0mm, B.Cu at (95.8, 100.1)
- added U2: 74HC4066PW,118, easyeda2kicad:TSSOP-14_L5.0-W4.4-P0.65-LS6.4-BL, F.Cu at (71.4, 90.4)
- C15: value 100u/6.3/tant -> 22uF/25V; footprint Capacitor_Tantalum_SMD:CP_EIA-3528-21_Kemet-B -> Capacitor_SMD:C_1206_3216Metric
- C16: value 22n -> 1n
- C2: value 22uF/25V -> 10u/25V; footprint Capacitor_SMD:C_1206_3216Metric -> Capacitor_SMD:C_0603_1608Metric
- C7: value 100u/tht -> 100n; footprint Capacitor_THT:CP_Radial_D8.0mm_P5.00mm -> Capacitor_SMD:C_0402_1005Metric; moved to F.Cu
- J1: value B4P -> Conn_01x03; footprint Critbit_lib:B4P_MATRIXPWR -> teensy:CONN-TH_MR30-M
- J5: footprint Critbit_lib:2x10_smdthrough -> Critbit_lib:SAMTEC_HLE-110-02-F-DV-BE-A
- R10: value 2 -> 3k/0603
- R19: value 6k/0603 -> 3k; footprint Resistor_SMD:R_0603_1608Metric_Pad0.98x0.95mm_HandSolder -> Resistor_SMD:R_0402_1005Metric
- TP1: footprint TestPoint:TestPoint_Pad_D1.0mm -> Critbit_lib:Nano_testpad_0.5x1.0mm
- moved J1 62.4 mm to (41.6, 103.7)
- moved C7 40.3 mm to (67.9, 88.1), turned to 90 degrees
- moved R31 24.8 mm to (73.2, 74.2), turned to -90 degrees
- moved R19 17.7 mm to (76.3, 90.8)
- moved C1 14.7 mm to (64.3, 58.7), turned to -90 degrees
- moved D2 12.8 mm to (108.0, 108.0)
- moved R32 12.8 mm to (104.8, 108.0)
- moved R13 12.5 mm to (92.2, 67.3)
- moved R3 11.0 mm to (92.2, 70.3), turned to 180 degrees
- moved R10 10.3 mm to (77.9, 67.2), turned to 180 degrees
- moved C2 9.79 mm to (86.8, 73.8), turned to 0 degrees
- moved R1 9.49 mm to (92.2, 68.8), turned to 0 degrees
- moved C41 9.19 mm to (91.6, 60.4)
- moved R27 9.14 mm to (90.0, 72.1), turned to 90 degrees
- moved R28 8.19 mm to (90.0, 70.2), turned to 90 degrees
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Connections:
- C16 pad 1: GND -> BAT
- C16 pad 2: BAT -> Net-(U8-SDRV)
- C7 pad 1: BAT -> GND
- C7 pad 2: GND -> 3V3_SYS
- D5 pad 1: Net-(D5-K) -> +VDC
- D5 pad 2: +VDC -> Net-(D5-A)
- J4 pad 3: /PWRBRD_TX -> /PROT_TX
- J4 pad 6: /I2C_INT -> /PROT_INT
- J4 pad 7: /SDA -> /PROT_SDA
- J4 pad 8: /SCL -> /PROT_SCL
- J5 pad 14: /I2C_INT -> /PROT_INT
- J5 pad 15: /PWRBRD_TX -> /PROT_TX
- J5 pad 16: /SDA -> /PROT_SDA
- J5 pad 18: /SCL -> /PROT_SCL
- R10 pad 1: GND -> Net-(JP1-A)
- R10 pad 2: /BQ_nCE -> Net-(U8-PROG)
- R19 pad 1: GND -> /OLED_RST
- R19 pad 2: Net-(U8-PROG) -> 3V3_SYS
- TP10 pad 1: /I2C_INT -> /PROT_INT
- TP15 pad 1: Net-(D5-K) -> Net-(D5-A)
- TP3 pad 1: Net-(D5-K) -> Net-(D5-A)
- TP8 pad 1: /SDA -> /PROT_SDA
- TP9 pad 1: /SCL -> /PROT_SCL
- U12 pad 10: /BQ_nCE -> GND
- U12 pad 11: /OLED_RST -> unconnected-(U12-PA5-Pad11)
- U8 pad 13: /BQ_nCE -> GND
- U8 pad 24: BAT -> Net-(U8-SDRV)
Routing:
- net /I2C_INT: track 106.9 -> 60.4 mm, vias 7 -> 4
- net /PROT_SCL: track 0.00 -> 46.4 mm, vias 0 -> 6
- net /SDA: track 109.2 -> 66.0 mm, vias 7 -> 4
- net /SCL: track 105.0 -> 63.1 mm, vias 7 -> 3
- net /PROT_SDA: track 0.00 -> 40.7 mm, vias 0 -> 6
- net /PROT_INT: track 0.00 -> 40.6 mm, vias 0 -> 5
- net /PWRBRD_TX: track 54.7 -> 17.2 mm, vias 5 -> 2
- net GND: track 173.8 -> 136.7 mm, vias 80 -> 69
- net /PROT_TX: track 0.00 -> 29.4 mm, vias 0 -> 4
- net VPWR: track 34.1 -> 5.27 mm, vias 10 -> 5
- net /3V3_ENA: track 40.0 -> 62.7 mm, vias 4 -> 5
- net /OLED_RST: track 23.8 -> 3.20 mm, vias 3 -> 1
- net /LIPO_NTC: track 56.5 -> 40.6 mm, vias 4 -> 3
- net VBUS: track 52.5 -> 36.9 mm
- net /PY32_ADC: track 12.6 -> 22.4 mm, vias 0 -> 2
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- removed copper zone on B.Cu, net SYS
Other:
- board text added: "1s"
- board text added: "2s"
- board text added: "3s"
- board text added: "Open:"
- board text added: "for @clue.lamp"
- board text added: "i2current 01/25"
- board text removed: "Rprog"
- board text removed: "Rprog: 3K->1S 6K->2S 10.5K->3S 17.4K->4S"
- board text removed: "i2current 01/25 for @clue.lamp"
