File: i2current.kicad_pcb (KiCad board)
At the start: 2 copper layers, 50 x 64 mm, 157 parts, among them CN2 JL15EDGA-38108G01, J1 Conn_01x03, J2 USB_C_Receptacle_USB2.0, J4 Conn_01x12_MountingPin, J5 EXT_IFACE, Q1 AON7544, Q2 AON7544, Q3 AON7544, Q6 AON7544, SW6 SW_SPDT, U1 SPX3819M5-L-3-3, U11 TPS56637RPAR, U12 PY32F002AW15U6TR, U13 USBLC6-4SC6, U2 74HC4066PW,118, U4 FTC252010S4R7MBCA, U5 FUSB302B01MPX, U6 MT2492, U7 JLC_OLED, U8 BQ25792RQMR

Commit message: may order
Parts:
- removed J1: Conn_01x03, teensy:CONN-TH_MR30-M
- removed R45: 100, Resistor_SMD:R_0402_1005Metric
- removed REF**: PinHeader_1x03_P2.54mm_Horizontal, Connector_PinHeader_2.54mm:PinHeader_1x03_P2.54mm_Horizontal
- added R29: 3k, Resistor_SMD:R_0402_1005Metric, F.Cu at (74.6, 82.7)
- added SW1: B2, Button_Switch_SMD:SW_SPST_TL3342, F.Cu at (80.1, 83.4)
- added TP21: TestPoint, Critbit_lib:Nano_testpad_0.5x1.0mm, F.Cu at (65.0, 100.0)
- added TP22: TestPoint, Critbit_lib:Nano_testpad_0.5x1.0mm, F.Cu at (66.1, 99.1)
- H1, H2, H3, H4: footprint MountingHole:MountingHole_3.2mm_M3_DIN965_Pad -> Critbit_lib:MountingHole_3.2mm_LONGE
- moved D2 14.2 mm to (94.8, 102.7)
- moved R32 14.1 mm to (91.8, 102.7)
- moved TP18 1.95 mm to (63.0, 63.8), turned to -90 degrees
- moved TP19 1.95 mm to (63.0, 63.8), turned to 90 degrees
- moved C1 1.57 mm to (64.3, 60.3)
- moved C46 0.39 mm to (72.3, 80.5)
- moved R40 0.35 mm to (70.4, 80.5)
- moved R14 0.30 mm to (75.2, 80.9)
- moved R22 0.30 mm to (74.1, 80.9)
- turned H4 to -135 degrees
- turned D5 to 180 degrees
- turned H1 to 45 degrees
- turned H2 to -45 degrees
- turned H3 to 135 degrees
- turned R41 to 0 degrees
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Connections:
- D13 pad 2: 3V3_SYS -> /PY32_HB_LED
- J4 pad 1: /GLOB_~{OFF} -> unconnected-(J4-Pin_1-Pad1)
- R22 pad 1: Net-(U12-PA6) -> Net-(U12-PA5)
- R40 pad 1: /PWRBRD_BOOT -> GND
- U12 pad 10: GND -> /PY32_BUT
- U12 pad 11: unconnected-(U12-PA5-Pad11) -> Net-(U12-PA5)
- U12 pad 12: Net-(U12-PA6) -> /PY32_HB_LED
Routing:
- net /PY32_BUT: track 0.00 -> 22.8 mm
- net GND: track 136.7 -> 154.8 mm, vias 69 -> 83
- net Net-(U12-PA5): track 0.00 -> 11.7 mm
- net Net-(U12-PA6): track 9.00 -> 0.00 mm
- net Net-(D5-A): track 0.00 -> 5.96 mm, vias 0 -> 1
- net +VDC: track 25.2 -> 19.2 mm, vias 3 -> 2
- net /PY32_HB_LED: track 0.00 -> 5.05 mm
- net VMCU: track 20.5 -> 25.5 mm, vias 5 -> 6
- net SYS: track 66.0 -> 70.9 mm
- net /PROT_SCL: track 46.4 -> 43.6 mm, vias 6 -> 4
- net BAT: track 7.86 -> 10.4 mm
- net /GLOB_~{OFF}: track 127.0 -> 124.5 mm, vias 9 -> 8
- net /SDA: track 66.0 -> 63.7 mm
- net Net-(JP2-A): track 7.51 -> 5.40 mm
- net /3V3_ENA: track 62.7 -> 64.8 mm, vias 5 -> 6
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- removed copper zone on F.Cu, net /5V_L
Other:
- outline, holes or cut-outs redrawn
- board text added: "Proudly sponsored by @clue.lamp"
- board text added: "github.com/ cr1tbit/ i2current"
- board text removed: "CPwr"
- board text removed: "Ts"
- board text removed: "for @clue.lamp"
- board text removed: "pwr"
- board text removed: "sys"
- board text removed: "usb"
